File: KiCad/RS/RS.kicad_pcb (KiCad board)
At the start: 2 copper layers, 179 parts, among them J1 XY2500V-B(5.0)-2P, J2 Screw_Terminal_01x12, J3 ST-LINK, J4 SPI, J5 MODEM, J6 I2C, J7 GNSS, J8 SIM, J9 ANTENNA, Q1 AO3400A, Q10 BC817, Q11 BC817, Q12 BC817, Q2 BC817, Q3 BC817, Q4 BC817, Q5 P60V/2A, Q6 P60V/2A, Q7 BC817, Q8 BC817, Q9 BC817, SW1 SW_Push, U1 MCP1700T-3302E/TT, U10 ST87M01-1301, U11 LDK320M-R, U2 LM2596S-5, U3 STM32C562KET6, U4 TLP185, U5 RV-3028-C7, U6 TLP185, U7 TLP185, U8 LD39050PUR, U9 EMIF03-SIM02M8, Y1 24MHz CL=8pF ESR=50Ω

Commit message: ADD: RF connections.
Parts:
- added JP1: Jumper_3_Bridged12, Connector_PinHeader_2.54mm:PinHeader_1x03_P2.54mm_Vertical, F.Cu at (94.3, 32.3)
- added JP2: Jumper_3_Bridged12, Connector_PinHeader_2.54mm:PinHeader_1x03_P2.54mm_Vertical, F.Cu at (98.9, 32.3)
- added L2: 1kΩ/100MHz, Inductor_SMD:L_0805_2012Metric_Pad1.05x1.20mm_HandSolder, F.Cu at (70.0, 39.4)
- added L3: 120Ω/100MHz/2A, Inductor_SMD:L_0805_2012Metric_Pad1.05x1.20mm_HandSolder, F.Cu at (70.0, 44.9)
- added L4: 120Ω/100MHz/2A, Inductor_SMD:L_0805_2012Metric_Pad1.05x1.20mm_HandSolder, F.Cu at (70.0, 47.6)
- added L5: 120Ω/100MHz/2A, Inductor_SMD:L_0805_2012Metric_Pad1.05x1.20mm_HandSolder, F.Cu at (70.0, 50.4)
- added L6: 120Ω/100MHz/2A, Inductor_SMD:L_0805_2012Metric_Pad1.05x1.20mm_HandSolder, F.Cu at (70.0, 53.1)
- moved C35 65.5 mm to (109.0, 50.0), turned to 90 degrees
- moved C33 65.5 mm to (86.0, 47.5), turned to -90 degrees
- moved C32 60.8 mm to (91.5, 48.0), turned to -90 degrees
- moved U10 35.8 mm to (93.0, 57.4)
- moved J9 29.3 mm to (97.0, 47.5)
- moved L7 3.61 mm to (107.5, 50.5)
- moved C34 1.00 mm to (106.0, 51.0)
- moved J7 1.00 mm to (106.0, 47.5)
Routing:
- net Net-(U10B-GNSS_ANT): track 0.00 -> 10.5 mm
- net Net-(U10B-VPA): track 0.00 -> 8.01 mm
- net Net-(J9-SIG): track 0.00 -> 2.48 mm
- net Net-(J7-SIG): track 0.00 -> 2.39 mm
- net VANT: track 0.00 -> 1.02 mm

Commit message: FIX: 0805 to 0402, modem leds+drivers
ADD: Modem part completed!
Parts:
- removed R67, R68, R69: 100k, Resistor_SMD:R_0805_2012Metric_Pad1.20x1.40mm_HandSolder
- J9: value ANTENNA -> ANT.
- R10, R16, R17, R23, R25, R29, R3, R4, R40, R41, R44, R45, R46, R47, R48, R49, R5, R52, R53, R54, R55, R56, R57: footprint Resistor_SMD:R_0805_2012Metric_Pad1.20x1.40mm_HandSolder -> Resistor_SMD:R_0402_1005Metric_Pad0.72x0.64mm_HandSolder
- R2, R27, R32, R33, R50, R51: value 470R -> 470
- R59, R60, R61: value 470R -> 50Ω; footprint Resistor_SMD:R_0805_2012Metric_Pad1.20x1.40mm_HandSolder -> Resistor_SMD:R_0402_1005Metric_Pad0.72x0.64mm_HandSolder
- R63, R64, R65: value 4k7 -> 2k2; footprint Resistor_SMD:R_0805_2012Metric_Pad1.20x1.40mm_HandSolder -> Resistor_SMD:R_0402_1005Metric_Pad0.72x0.64mm_HandSolder
- R66: value 10k -> 10kΩ
- moved D19 323.1 mm to (156.0, 39.8)
- moved J1 319.1 mm to (148.8, 81.3)
- moved D18 317.5 mm to (151.0, 39.8)
- moved R66 314.4 mm to (156.2, 31.1), turned to -90 degrees
- moved R60 313.9 mm to (150.2, 41.4)
- moved R61 312.5 mm to (155.2, 41.4)
- moved R65 312.0 mm to (154.6, 43.2), turned to -90 degrees
- moved D17 312.0 mm to (146.0, 39.8)
- moved R62 310.8 mm to (153.2, 30.2)
- moved C26 310.0 mm to (148.6, 36.7), turned to 180 degrees
- moved R59 308.6 mm to (145.2, 41.4)
- moved R64 307.0 mm to (149.6, 43.2), turned to -90 degrees
- moved R63 302.0 mm to (144.6, 43.2), turned to -90 degrees
- moved C36 296.7 mm to (154.0, 27.2), turned to -90 degrees
- moved C25 295.6 mm to (147.9, 32.4), turned to 180 degrees
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Routing:
- net VMOD: track 0.00 -> 54.0 mm
- net Net-(Q9-C): track 0.00 -> 30.5 mm, vias 0 -> 2
- net DCDC_EN: track 0.00 -> 24.6 mm, vias 0 -> 2
- net VRFFE: track 0.00 -> 19.9 mm, vias 0 -> 2
- net MODEM_LED1: track 0.00 -> 16.8 mm, vias 0 -> 2
- net Net-(U10C-GPIO_01): track 0.00 -> 16.4 mm, vias 0 -> 2
- net Net-(U10C-GPIO_02): track 0.00 -> 15.7 mm, vias 0 -> 2
- net Net-(U10C-GPIO_00): track 0.00 -> 15.3 mm, vias 0 -> 2
- net MODEM_LED0: track 0.00 -> 12.5 mm, vias 0 -> 2
- net Net-(J8-RST): track 0.00 -> 12.0 mm
- net VANT: track 1.02 -> 9.73 mm
- net Net-(J8-CLK): track 0.00 -> 8.02 mm
- net GND: track 0.00 -> 7.53 mm, vias 0 -> 2
- net VSIM: track 0.00 -> 7.07 mm
- net Net-(U10A-VPMU_2): track 0.00 -> 6.43 mm
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- added copper zone on B.Cu, net GND
- added copper zone on F.Cu, net GND
Other:
- board outline added: 50 x 80 mm

Commit message: ADD: New PCB.
Parts:
- added C37: 100n, Capacitor_SMD:C_0402_1005Metric_Pad0.74x0.62mm_HandSolder, F.Cu at (215.7, 52.6)
- added C38: 10μ/10V, Capacitor_SMD:C_0402_1005Metric_Pad0.74x0.62mm_HandSolder, F.Cu at (215.7, 54.5)
- added C39: 1n, Inductor_SMD:L_0402_1005Metric_Pad0.77x0.64mm_HandSolder, F.Cu at (171.3, 52.6)
- added C40: 33p, Capacitor_SMD:C_0402_1005Metric_Pad0.74x0.62mm_HandSolder, F.Cu at (215.7, 56.5)
- added C41: 1μ/10V, Capacitor_SMD:C_0402_1005Metric_Pad0.74x0.62mm_HandSolder, F.Cu at (215.7, 58.5)
- added L8: 100nH, Inductor_SMD:L_0402_1005Metric, F.Cu at (197.6, 98.3)
- added Q13: BC817, Package_TO_SOT_SMD:SOT-23, F.Cu at (208.1, 83.5)
- added Q14: BC817, Package_TO_SOT_SMD:SOT-23, F.Cu at (208.1, 88.0)
- added R67: 1k, Resistor_SMD:R_0402_1005Metric_Pad0.72x0.64mm_HandSolder, F.Cu at (184.4, 58.6)
- added R68: 1k, Resistor_SMD:R_0402_1005Metric_Pad0.72x0.64mm_HandSolder, F.Cu at (184.4, 60.5)
- added R69: 1k, Resistor_SMD:R_0402_1005Metric_Pad0.72x0.64mm_HandSolder, F.Cu at (184.4, 62.5)
- added R70: 10k 0.1%, Resistor_SMD:R_0402_1005Metric_Pad0.72x0.64mm_HandSolder, F.Cu at (184.4, 64.5)
- C1: value 1μ/50V -> 100n/50V; footprint Capacitor_SMD:C_0805_2012Metric_Pad1.18x1.45mm_HandSolder -> Capacitor_SMD:C_0402_1005Metric_Pad0.74x0.62mm_HandSolder
- C10: value 100n -> 47μ/10V
- C11: value 12p -> 100n; footprint Capacitor_SMD:C_0805_2012Metric_Pad1.18x1.45mm_HandSolder -> Capacitor_SMD:C_0402_1005Metric_Pad0.74x0.62mm_HandSolder
- C12: value 12p -> 1μ/10V; footprint Capacitor_SMD:C_0805_2012Metric_Pad1.18x1.45mm_HandSolder -> Capacitor_SMD:C_0402_1005Metric_Pad0.74x0.62mm_HandSolder
- C13: value 1n -> 100n; footprint Capacitor_SMD:C_0805_2012Metric_Pad1.18x1.45mm_HandSolder -> Capacitor_SMD:C_0402_1005Metric_Pad0.74x0.62mm_HandSolder
- C14, C21, C23, C24, C25, C27, C29, C31: footprint Capacitor_SMD:C_0805_2012Metric_Pad1.18x1.45mm_HandSolder -> Capacitor_SMD:C_0402_1005Metric_Pad0.74x0.62mm_HandSolder
- C15: value 1μ/50V -> 12p; footprint Capacitor_SMD:C_0805_2012Metric_Pad1.18x1.45mm_HandSolder -> Capacitor_SMD:C_0402_1005Metric_Pad0.74x0.62mm_HandSolder
- C16: value 2μ2/10V -> 12p; footprint Capacitor_SMD:C_0805_2012Metric_Pad1.18x1.45mm_HandSolder -> Capacitor_SMD:C_0402_1005Metric_Pad0.74x0.62mm_HandSolder
- C17: value 100n -> 1n; footprint Capacitor_SMD:C_0805_2012Metric_Pad1.18x1.45mm_HandSolder -> Inductor_SMD:L_0402_1005Metric_Pad0.77x0.64mm_HandSolder
- C18, C26, C28, C33: value 10μ/10V -> 100n; footprint Capacitor_SMD:C_1206_3216Metric_Pad1.33x1.80mm_HandSolder -> Capacitor_SMD:C_0402_1005Metric_Pad0.74x0.62mm_HandSolder
- C19: value 100n -> 1μ/10V; footprint Capacitor_SMD:C_0805_2012Metric_Pad1.18x1.45mm_HandSolder -> Capacitor_SMD:C_0402_1005Metric_Pad0.74x0.62mm_HandSolder
- C2: value 470u/50V -> 10μ/50V; footprint Capacitor_THT:CP_Radial_D12.5mm_P5.00mm -> Capacitor_SMD:C_1210_3225Metric_Pad1.33x2.70mm_HandSolder
- C20: value 100n -> 2μ2/10V; footprint Capacitor_SMD:C_0805_2012Metric_Pad1.18x1.45mm_HandSolder -> Capacitor_SMD:C_0402_1005Metric_Pad0.74x0.62mm_HandSolder
- C22, C32, C7, C9: value 100n -> 10μ/10V; footprint Capacitor_SMD:C_0805_2012Metric_Pad1.18x1.45mm_HandSolder -> Capacitor_SMD:C_0402_1005Metric_Pad0.74x0.62mm_HandSolder
- C3: value 1μ/50V -> 10μ/50V; footprint Capacitor_SMD:C_0805_2012Metric_Pad1.18x1.45mm_HandSolder -> Capacitor_SMD:C_1210_3225Metric_Pad1.33x2.70mm_HandSolder
- C30: footprint Capacitor_SMD:C_1206_3216Metric_Pad1.33x1.80mm_HandSolder -> Capacitor_SMD:C_0402_1005Metric_Pad0.74x0.62mm_HandSolder
- C34: value 1n -> 10μ/10V; footprint Capacitor_SMD:C_0402_1005Metric -> Capacitor_SMD:C_0402_1005Metric_Pad0.74x0.62mm_HandSolder
- C35: value 33p -> 100n; footprint Capacitor_SMD:C_0402_1005Metric -> Capacitor_SMD:C_0402_1005Metric_Pad0.74x0.62mm_HandSolder
- C36, C8: value 1μ/50V -> 10μ/10V; footprint Capacitor_SMD:C_0805_2012Metric_Pad1.18x1.45mm_HandSolder -> Capacitor_SMD:C_0402_1005Metric_Pad0.74x0.62mm_HandSolder
- C4: value 47μ/10V -> 100n/50V; footprint Capacitor_SMD:C_0805_2012Metric_Pad1.18x1.45mm_HandSolder -> Capacitor_SMD:C_0402_1005Metric_Pad0.74x0.62mm_HandSolder
- C5: value 470u/16V -> 75pF/50V; footprint Capacitor_THT:CP_Radial_D8.0mm_P3.50mm -> Capacitor_SMD:C_0402_1005Metric_Pad0.74x0.62mm_HandSolder
- C6: value 470u/16V -> 100n/50V; footprint Capacitor_THT:CP_Radial_D8.0mm_P3.50mm -> Capacitor_SMD:C_0402_1005Metric_Pad0.74x0.62mm_HandSolder
- D1: value LED red -> SMAJ26A; footprint Diode_SMD:D_0805_2012Metric_Pad1.15x1.40mm_HandSolder -> Diode_SMD:D_SMA
- D11, D12: footprint Diode_SMD:D_MiniMELF -> Diode_SMD:D_SOD-323
- D15, D16, D6: value LED amber -> LED orange
- D3: value SS56 -> LED red; footprint Diode_SMD:D_SMA_Handsoldering -> Diode_SMD:D_0805_2012Metric_Pad1.15x1.40mm_HandSolder
- D4: value 3V3 -> 1V; footprint Diode_SMD:D_SOD-523 -> Diode_SMD:D_SMA_Handsoldering
- J1: value XY2500V-B(5.0)-2P -> 4.5-28V; footprint Connector_Phoenix_MSTB:PhoenixContact_MSTBVA_2,5_2-G_1x02_P5.00mm_Vertical -> Connector_Phoenix_MC:PhoenixContact_MCV_1,5_2-G-3.81_1x02_P3.81mm_Vertical
- L1: value 68μH/3.9A -> 15μH/2.05A; footprint Inductor_SMD:L_Coilcraft_MSS1278T-XXX -> Inductor_SMD:L_Cenker_CKCS6045
- L2, L3, L4, L5, L6: footprint Inductor_SMD:L_0805_2012Metric_Pad1.05x1.20mm_HandSolder -> Inductor_SMD:L_0402_1005Metric_Pad0.77x0.64mm_HandSolder
- L7: value 100nH -> 120Ω/100MHz/2A; footprint Inductor_SMD:L_0402_1005Metric -> Inductor_SMD:L_0402_1005Metric_Pad0.77x0.64mm_HandSolder
- R1: value 1k -> 49R9; footprint Resistor_SMD:R_0805_2012Metric_Pad1.20x1.40mm_HandSolder -> Resistor_SMD:R_0402_1005Metric_Pad0.72x0.64mm_HandSolder
- R10, R17: value 10k -> 0R; footprint Resistor_SMD:R_0402_1005Metric_Pad0.72x0.64mm_HandSolder -> Resistor_SMD:R_0805_2012Metric_Pad1.20x1.40mm_HandSolder
- R11: value 2k -> 0R
- R13: value 2k -> 10k; footprint Resistor_SMD:R_0805_2012Metric_Pad1.20x1.40mm_HandSolder -> Resistor_SMD:R_0402_1005Metric_Pad0.72x0.64mm_HandSolder
- R14: value 0R -> 2k; footprint Resistor_SMD:R_0805_2012Metric_Pad1.20x1.40mm_HandSolder -> Resistor_SMD:R_0402_1005Metric_Pad0.72x0.64mm_HandSolder
- R16: value 10k -> 2k
- R19, R26: value 200 -> 10k; footprint Resistor_SMD:R_0805_2012Metric_Pad1.20x1.40mm_HandSolder -> Resistor_SMD:R_0402_1005Metric_Pad0.72x0.64mm_HandSolder
- R2: value 470 -> 180; footprint Resistor_SMD:R_0805_2012Metric_Pad1.20x1.40mm_HandSolder -> Resistor_SMD:R_0402_1005Metric_Pad0.72x0.64mm_HandSolder
- R20: value 68k 0.1% -> 10k; footprint Resistor_SMD:R_0805_2012Metric_Pad1.20x1.40mm_HandSolder -> Resistor_SMD:R_0402_1005Metric_Pad0.72x0.64mm_HandSolder
- R21: value 1k -> 0R
- R22: value 133R 0.1% -> 120; footprint Resistor_SMD:R_0805_2012Metric_Pad1.20x1.40mm_HandSolder -> Resistor_SMD:R_0402_1005Metric_Pad0.72x0.64mm_HandSolder
- R23: value 10k -> 68k 0.1%; footprint Resistor_SMD:R_0402_1005Metric_Pad0.72x0.64mm_HandSolder -> Resistor_SMD:R_0805_2012Metric_Pad1.20x1.40mm_HandSolder
- R24: value 100 -> 120; footprint Resistor_SMD:R_0805_2012Metric_Pad1.20x1.40mm_HandSolder -> Resistor_SMD:R_0402_1005Metric_Pad0.72x0.64mm_HandSolder
- R25: value 4k7 -> 133 0.1%; footprint Resistor_SMD:R_0402_1005Metric_Pad0.72x0.64mm_HandSolder -> Resistor_SMD:R_0805_2012Metric_Pad1.20x1.40mm_HandSolder
- R27: value 470 -> 120; footprint Resistor_SMD:R_0805_2012Metric_Pad1.20x1.40mm_HandSolder -> Resistor_SMD:R_0402_1005Metric_Pad0.72x0.64mm_HandSolder
- R28: value 27.7k 0.1% -> 4k7; footprint Resistor_SMD:R_0805_2012Metric_Pad1.20x1.40mm_HandSolder -> Resistor_SMD:R_0402_1005Metric_Pad0.72x0.64mm_HandSolder
- R29: value 4k7 -> 200
- R3, R52, R53: value 10k -> 82
- R30: value 100k -> 82; footprint Resistor_SMD:R_0805_2012Metric_Pad1.20x1.40mm_HandSolder -> Resistor_SMD:R_0402_1005Metric_Pad0.72x0.64mm_HandSolder
- R31: value 100k -> 27.7k 0.1%
- R32: value 470 -> 4k7; footprint Resistor_SMD:R_0805_2012Metric_Pad1.20x1.40mm_HandSolder -> Resistor_SMD:R_0402_1005Metric_Pad0.72x0.64mm_HandSolder
- R33: value 470 -> 100k; footprint Resistor_SMD:R_0805_2012Metric_Pad1.20x1.40mm_HandSolder -> Resistor_SMD:R_0402_1005Metric_Pad0.72x0.64mm_HandSolder
- R34, R35: value 3k3/0.4W -> 180; footprint Resistor_SMD:R_0805_2012Metric_Pad1.20x1.40mm_HandSolder -> Resistor_SMD:R_0402_1005Metric_Pad0.72x0.64mm_HandSolder
- R36, R37: value 22k -> 1.8k 0.5W; footprint Resistor_SMD:R_0805_2012Metric_Pad1.20x1.40mm_HandSolder -> Resistor_SMD:R_0603_1608Metric_Pad0.98x0.95mm_HandSolder
- R38, R39: value 47k -> 1k; footprint Resistor_SMD:R_0805_2012Metric_Pad1.20x1.40mm_HandSolder -> Resistor_SMD:R_0402_1005Metric_Pad0.72x0.64mm_HandSolder
- R4: value 4k7 -> 100k
- R40, R41: value 4k7 -> 47k
- R42, R43: value 1k -> 4k7; footprint Resistor_SMD:R_0805_2012Metric_Pad1.20x1.40mm_HandSolder -> Resistor_SMD:R_0402_1005Metric_Pad0.72x0.64mm_HandSolder
- R44, R45, R57: value 4k7 -> 1k
- R48, R49: value 10k -> 4k7
- R5: value 4k7 -> 13k3
- R50, R51: value 470 -> 10k; footprint Resistor_SMD:R_0805_2012Metric_Pad1.20x1.40mm_HandSolder -> Resistor_SMD:R_0402_1005Metric_Pad0.72x0.64mm_HandSolder
- R54: value 51k -> 0R; footprint Resistor_SMD:R_0402_1005Metric_Pad0.72x0.64mm_HandSolder -> Resistor_SMD:R_0805_2012Metric_Pad1.20x1.40mm_HandSolder
- R55: value 24k -> 51k 0.1%
- R56: value 10k -> 24k 0.1%
- R58: value 100k -> 1k; footprint Resistor_SMD:R_0805_2012Metric_Pad1.20x1.40mm_HandSolder -> Resistor_SMD:R_0402_1005Metric_Pad0.72x0.64mm_HandSolder
- R59, R60: value 50Ω -> 4k7
- R6: value 0R -> 10k; footprint Resistor_SMD:R_0805_2012Metric_Pad1.20x1.40mm_HandSolder -> Resistor_SMD:R_0402_1005Metric_Pad0.72x0.64mm_HandSolder
- R61: value 50Ω -> 1k
- R62: value 18k -> 4k7; footprint Resistor_SMD:R_0805_2012Metric_Pad1.20x1.40mm_HandSolder -> Resistor_SMD:R_0402_1005Metric_Pad0.72x0.64mm_HandSolder
- R63, R64, R65: value 2k2 -> 180
- R66: value 10kΩ -> 18k 0.1%; footprint Resistor_SMD:R_0805_2012Metric_Pad1.20x1.40mm_HandSolder -> Resistor_SMD:R_0402_1005Metric_Pad0.72x0.64mm_HandSolder
- R7, R8: value 0R -> 4k7; footprint Resistor_SMD:R_0805_2012Metric_Pad1.20x1.40mm_HandSolder -> Resistor_SMD:R_0402_1005Metric_Pad0.72x0.64mm_HandSolder
- U2: value LM2596S-5 -> TPS54202; footprint Package_TO_SOT_SMD:TO-263-5_TabPin3 -> Package_TO_SOT_SMD:SOT-23-6
- moved J4 317.1 mm to (241.1, 31.3)
- moved R10 294.5 mm to (212.9, 72.4)
- moved R9 294.5 mm to (212.9, 69.4)
- moved R11 294.2 mm to (212.9, 75.3)
- moved R12 294.2 mm to (212.9, 78.3)
- moved R15 293.0 mm to (212.9, 81.2)
- moved R21 292.8 mm to (212.9, 90.1)
- moved R17 292.5 mm to (212.9, 84.2)
- moved R18 292.5 mm to (212.9, 87.1)
- moved JP2 290.2 mm to (231.0, 100.5)
- moved R36 286.4 mm to (219.5, 55.6)
- moved R37 286.4 mm to (219.5, 58.1)
- moved TP4 269.6 mm to (188.3, 56.5)
- moved TP1 269.0 mm to (188.3, 51.9)
- moved TP10 269.0 mm to (192.9, 65.7)
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Connections:
- C1 pad 1: +24V -> Net-(U2-SW)
- C1 pad 2: GND -> Net-(U2-BOOT)
- C10 pad 1: GND -> +3V3
- C10 pad 2: +3V3 -> GND
- C11 pad 1: Net-(U3A-PH0-OSC_IN) -> GND
- C11 pad 2: GND -> Net-(U3A-VREF+)
- C12 pad 1: Net-(U3A-PH1-OSC_OUT) -> GND
- C12 pad 2: GND -> Net-(U3A-VREF+)
- C13 pad 2: Net-(U3B-PA1) -> +3V3
- C14 pad 2: NRST -> +3V3
- C15 pad 1: GND -> Net-(U3A-PH0-OSC_IN)
- C15 pad 2: Net-(U3B-PA0) -> GND
- C16 pad 1: GND -> Net-(U3A-PH1-OSC_OUT)
- C16 pad 2: Net-(U3A-VCAP) -> GND
- C17 pad 2: +3V3 -> Net-(U3B-PA1)
- C18 pad 2: Net-(U5-VBACKUP) -> NRST
- C19 pad 2: D_IN1_M -> Net-(U3B-PA0)
- C20 pad 2: D_IN2_M -> Net-(U3A-VCAP)
- C21 pad 2: Net-(D11-K) -> +3V3
- C22 pad 2: Net-(D12-K) -> Net-(U5-VBACKUP)
- C23 pad 1: GND -> D_IN1_M
- C23 pad 2: VSIM -> GND
- C24 pad 1: GND -> D_IN2_M
- C24 pad 2: VSIM -> GND
- C25 pad 1: GND -> Net-(D11-K)
- C25 pad 2: Net-(U10A-VPMU_1) -> GND
- C26 pad 1: GND -> Net-(D12-K)
- C26 pad 2: Net-(U10A-VPMU_1) -> GND
- C27 pad 2: Net-(U10A-VPMU_2) -> VSIM
- C28 pad 2: Net-(U10A-VPMU_2) -> VSIM
- C29 pad 2: Net-(U10A-VDCDC) -> Net-(U10A-VPMU_1)
- C3 pad 1: +5V -> +24V
- C30 pad 2: Net-(U10A-VDCDC) -> Net-(U10A-VPMU_1)
- C31 pad 2: +3V3 -> Net-(U10A-VPMU_2)
- C32 pad 2: Net-(U10B-VPA) -> Net-(U10A-VPMU_2)
- C33 pad 2: Net-(U10B-VPA) -> Net-(U10A-VDCDC)
- C34 pad 1: Net-(J7-SIG) -> GND
- C34 pad 2: Net-(U10B-GNSS_ANT) -> Net-(U10A-VDCDC)
- C35 pad 1: VANT -> GND
- C35 pad 2: GND -> VMOD_VIO
- C36 pad 1: VANT -> GND
- C36 pad 2: GND -> VMOD_VIO
- C4 pad 1: +3V3 -> +24V
- C5 pad 1: +5V -> Net-(C5-Pad1)
- C5 pad 2: GND -> Net-(U2-FB)
- C7 pad 1: GND -> +5V
- C7 pad 2: Net-(U3A-VREF+) -> GND
- C8 pad 1: GND -> +5V
- C8 pad 2: Net-(U3A-VREF+) -> GND
- C9 pad 1: GND -> +5V
- C9 pad 2: +3V3 -> GND
- D1 pad 1: GND -> +24V
- D1 pad 2: Net-(D1-A) -> GND
- D17 pad 2: +3V3 -> +5V
- D18 pad 2: +3V3 -> +5V
- D19 pad 2: +3V3 -> +5V
- D3 pad 1: Net-(D3-K) -> GND
- D3 pad 2: GND -> Net-(D3-A)
- L1 pad 1: Net-(D3-K) -> Net-(U2-SW)
- L6 pad 2: Net-(U10B-VPA) -> VMOD_VIO
- L7 pad 1: Net-(J7-SIG) -> VMOD
- L7 pad 2: VANT -> Net-(U10B-VPA)
- R1 pad 2: Net-(D1-A) -> Net-(C5-Pad1)
- R10 pad 1: +3V3 -> MODEM_RST
- R10 pad 2: NRST -> Net-(U3B-PB8-BOOT0)
- R11 pad 1: ADC -> Net-(U3B-PA12)
- R11 pad 2: Net-(U3B-PA0) -> X_MODEM_RX
- R12 pad 1: Net-(U3B-PA12) -> Net-(U3B-PA11)
- R12 pad 2: MODEM_RX -> X_MODEM_TX
- R13 pad 1: RCS -> +3V3
- R13 pad 2: Net-(U3B-PA1) -> NRST
- R14 pad 1: Net-(U3B-PA11) -> ADC
- R14 pad 2: MODEM_TX -> Net-(U3B-PA0)
- R15 pad 1: Net-(U3B-PA7) -> Net-(U3B-PA12)
- R15 pad 2: MODEM_WAKE_UP -> MODEM_RX
- R16 pad 1: SPI_MISO -> RCS
- R16 pad 2: GND -> Net-(U3B-PA1)
- R17 pad 1: SPI_IRQ -> Net-(U3B-PA11)
- R17 pad 2: GND -> MODEM_TX
- R18 pad 1: X_MODEM_WAKE_UP -> Net-(U3B-PA7)
- R18 pad 2: Net-(U3B-PA7) -> MODEM_WAKE_UP
- R19 pad 1: +3V3 -> SPI_MISO
- R19 pad 2: Net-(R19-Pad2) -> GND
- R2 pad 1: +3V3 -> +5V
- R20 pad 1: Net-(R20-Pad1) -> SPI_IRQ
- R20 pad 2: A_IN -> GND
- R21 pad 1: Net-(R20-Pad1) -> X_MODEM_WAKE_UP
- R21 pad 2: ADC -> Net-(U3B-PA7)
- R22 pad 1: Net-(Q1-D) -> +3V3
- R22 pad 2: Net-(R20-Pad1) -> Net-(R22-Pad2)
- R23 pad 1: RTC_EVI -> Net-(R23-Pad1)
- R23 pad 2: GND -> A_IN
- R24 pad 1: GND -> Net-(R23-Pad1)
- R24 pad 2: RCS -> ADC
- R25 pad 1: +3V3 -> Net-(Q1-D)
- R25 pad 2: Net-(Q2-C) -> Net-(R23-Pad1)
- R26 pad 1: Net-(Q2-C) -> RTC_EVI
- R26 pad 2: Net-(Q1-G) -> GND
- R27 pad 1: VM -> GND
- R27 pad 2: Net-(D6-A) -> RCS
- R28 pad 1: GND -> +3V3
- R28 pad 2: Net-(R20-Pad1) -> Net-(Q2-C)
- R29 pad 1: VM -> Net-(Q2-C)
- R29 pad 2: Net-(Q2-B) -> Net-(Q1-G)
- R3 pad 1: +3V3 -> Net-(D3-A)
- R3 pad 2: SPI_NSS -> +3V3
- R30 pad 1: Net-(Q1-G) -> VM
- R30 pad 2: GND -> Net-(D6-A)
- R31 pad 1: Net-(Q2-B) -> GND
- R31 pad 2: GND -> Net-(R23-Pad1)
- R32 pad 1: +3V3 -> VM
- R32 pad 2: Net-(D7-A) -> Net-(Q2-B)
- R33 pad 1: +3V3 -> Net-(Q1-G)
- R33 pad 2: Net-(D8-A) -> GND
- R34 pad 1: D_IN1 -> +5V
- R34 pad 2: Net-(D9-K) -> Net-(D7-A)
- R35 pad 1: D_IN2 -> +5V
- R35 pad 2: Net-(D10-K) -> Net-(D8-A)
- R36 pad 1: D_IN1_M -> D_IN1
- R36 pad 2: Net-(Q3-B) -> Net-(D9-K)
- R37 pad 1: D_IN2_M -> D_IN2
- R37 pad 2: Net-(Q4-B) -> Net-(D10-K)
- R38 pad 2: GND -> Net-(Q3-B)
- R39 pad 2: GND -> Net-(Q4-B)
- R4 pad 1: +3V3 -> Net-(C5-Pad1)
- R4 pad 2: I2C_SCL -> Net-(U2-FB)
- R40 pad 1: Net-(D11-K) -> D_IN1_M
- R40 pad 2: Net-(D11-A) -> GND
- R41 pad 1: Net-(D12-K) -> D_IN2_M
- R41 pad 2: Net-(D12-A) -> GND
- R42 pad 1: Net-(D11-A) -> Net-(D11-K)
- R42 pad 2: Net-(Q5-G) -> Net-(D11-A)
- R43 pad 1: Net-(D12-A) -> Net-(D12-K)
- R43 pad 2: Net-(Q6-G) -> Net-(D12-A)
- R44 pad 2: Net-(Q7-C) -> Net-(Q5-G)
- R45 pad 2: Net-(Q8-C) -> Net-(Q6-G)
- R46 pad 1: D_OUT1_M -> Net-(D11-A)
- R46 pad 2: Net-(Q7-B) -> Net-(Q7-C)
- R47 pad 1: D_OUT2_M -> Net-(D12-A)
- R47 pad 2: Net-(Q8-B) -> Net-(Q8-C)
- R48 pad 1: D_OUT1 -> D_OUT1_M
- R48 pad 2: GND -> Net-(Q7-B)
- R49 pad 1: D_OUT2 -> D_OUT2_M
- R49 pad 2: GND -> Net-(Q8-B)
- R5 pad 1: +3V3 -> GND
- R5 pad 2: I2C_SDA -> Net-(U2-FB)
- R50 pad 1: D_OUT1_M -> D_OUT1
- R50 pad 2: Net-(D15-A) -> GND
- R51 pad 1: D_OUT2_M -> D_OUT2
- R51 pad 2: Net-(D16-A) -> GND
- R52 pad 1: Net-(Q7-B) -> Net-(D15-A)
- R52 pad 2: GND -> D_OUT1_M
- R53 pad 1: Net-(Q8-B) -> Net-(D16-A)
- R53 pad 2: GND -> D_OUT2_M
- R54 pad 1: VMOD -> Net-(U8-EN)
- R54 pad 2: Net-(U8-ADJ) -> +5V
- R55 pad 1: Net-(U8-ADJ) -> VMOD
- R55 pad 2: GND -> Net-(U8-ADJ)
- R56 pad 1: +3V3 -> Net-(U8-ADJ)
- R56 pad 2: Net-(Q9-C) -> GND
- R57 pad 1: MODEM_RST -> Net-(Q9-C)
- R57 pad 2: Net-(Q9-B) -> VMOD_VIO
- R58 pad 1: Net-(Q9-B) -> Net-(Q10-C)
- R58 pad 2: GND -> VMOD_VIO
- R59 pad 1: Net-(D17-K) -> Net-(Q10-C)
- R59 pad 2: Net-(Q10-C) -> Net-(Q9-B)
- R6 pad 1: Net-(U3B-PB8-BOOT0) -> +3V3
- R6 pad 2: X_MODEM_RST -> SPI_NSS
- R60 pad 1: Net-(D18-K) -> MODEM_WAKE_UP
- R60 pad 2: Net-(Q11-C) -> Net-(Q10-B)
- R61 pad 1: Net-(D19-K) -> Net-(Q11-C)
- R61 pad 2: Net-(Q12-C) -> VMOD_VIO
- R62 pad 1: VANT -> MODEM_RST
- R62 pad 2: Net-(U11-ADJ) -> Net-(Q11-B)
- R63 pad 1: DCDC_EN -> Net-(D17-K)
- R63 pad 2: Net-(Q10-B) -> Net-(Q12-C)
- R64 pad 1: MODEM_LED0 -> Net-(D18-K)
- R64 pad 2: Net-(Q11-B) -> Net-(Q13-C)
- R65 pad 1: MODEM_LED1 -> Net-(D19-K)
- R65 pad 2: Net-(Q12-B) -> Net-(Q14-C)
- R66 pad 1: Net-(U11-ADJ) -> VANT
- R66 pad 2: GND -> Net-(U11-ADJ)
- R7 pad 1: MODEM_RST -> +3V3
- R7 pad 2: Net-(U3B-PB8-BOOT0) -> I2C_SCL
- R8 pad 1: Net-(U3B-PA12) -> +3V3
- R8 pad 2: X_MODEM_RX -> I2C_SDA
- R9 pad 1: Net-(U3B-PA11) -> Net-(U3B-PB8-BOOT0)
- R9 pad 2: X_MODEM_TX -> X_MODEM_RST
- U10 pad 20: +3V3 -> VMOD_VIO
- U10 pad 38: Net-(Q9-C) -> Net-(Q11-C)
- U10 pad 39: MODEM_WAKE_UP -> Net-(Q9-C)
- U2 pad 1: +24V -> GND
- U2 pad 2: Net-(D3-K) -> Net-(U2-SW)
- U2 pad 3: GND -> +24V
- U2 pad 4: +5V -> Net-(U2-FB)
- U2 pad 5: GND -> unconnected-(U2-EN-Pad5)
- U4 pad 1: Net-(R19-Pad2) -> Net-(R22-Pad2)
- U4 pad 4: Net-(R20-Pad1) -> Net-(R23-Pad1)
- U8 pad 1: +5V -> Net-(U8-EN)
- U8 pad 6: +5V -> Net-(U8-EN)
Routing:
- net VMOD: track 54.0 -> 0.00 mm
- net Net-(Q9-C): track 30.5 -> 0.00 mm, vias 2 -> 0
- net DCDC_EN: track 24.6 -> 0.00 mm, vias 2 -> 0
- net VRFFE: track 19.9 -> 0.00 mm, vias 2 -> 0
- net MODEM_LED1: track 16.8 -> 0.00 mm, vias 2 -> 0
- net Net-(U10C-GPIO_01): track 16.4 -> 0.00 mm, vias 2 -> 0
- net Net-(U10C-GPIO_02): track 15.7 -> 0.00 mm, vias 2 -> 0
- net Net-(U10C-GPIO_00): track 15.3 -> 0.00 mm, vias 2 -> 0
- net MODEM_LED0: track 12.5 -> 0.00 mm, vias 2 -> 0
- net Net-(J8-RST): track 12.0 -> 0.00 mm
- net VANT: track 9.73 -> 0.00 mm
- net Net-(J8-CLK): track 8.02 -> 0.00 mm
- net Net-(U10B-GNSS_ANT): track 7.76 -> 0.00 mm
- net GND: track 7.53 -> 0.00 mm, vias 2 -> 0
- net Net-(U10B-VPA): track 7.29 -> 0.00 mm
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Other:
- board text added: "+"
- board text added: "-"
- board text added: "3V3"
- board text added: "5V"
- board text added: "ANALOG IN"
- board text added: "DIGITAL IN1"
- board text added: "DIGITAL IN2"
- board text added: "DIGITAL OUT1"
- board text added: "DIGITAL OUT2"
- board text added: "P+"
- board text added: "P-"
- board text added: "SIG"
- board text added: "VM"

Commit message: FIX: Everything. 1.0.
Parts:
- D1: footprint Diode_SMD:D_SMA -> CodeDog:D_SMA
- D10, D5, D9: footprint Diode_SMD:D_SOD-123 -> CodeDog:D_SOD-123
- D11, D12: footprint Diode_SMD:D_SOD-323 -> CodeDog:D_SOD-323
- D13, D14, D4: footprint Diode_SMD:D_SMA_Handsoldering -> CodeDog:D_SMA
- TP1: value Test Point -> GND; footprint Connector_PinHeader_2.54mm:PinHeader_1x01_P2.54mm_Vertical -> TestPoint:TestPoint_Keystone_5015_Micro_Mini
- TP10: value Test Point -> ADC; footprint Connector_PinHeader_2.54mm:PinHeader_1x01_P2.54mm_Vertical -> TestPoint:TestPoint_Keystone_5015_Micro_Mini
- TP11: value Test Point -> RCS; footprint Connector_PinHeader_2.54mm:PinHeader_1x01_P2.54mm_Vertical -> TestPoint:TestPoint_Keystone_5015_Micro_Mini
- TP12: value Test Point -> VM; footprint Connector_PinHeader_2.54mm:PinHeader_1x01_P2.54mm_Vertical -> TestPoint:TestPoint_Keystone_5015_Micro_Mini
- TP13: value Test Point -> D_IN1_M; footprint Connector_PinHeader_2.54mm:PinHeader_1x01_P2.54mm_Vertical -> TestPoint:TestPoint_Keystone_5015_Micro_Mini
- TP14: value Test Point -> D_IN2_M; footprint Connector_PinHeader_2.54mm:PinHeader_1x01_P2.54mm_Vertical -> TestPoint:TestPoint_Keystone_5015_Micro_Mini
- TP15: value Test Point -> D_OUT1_M; footprint Connector_PinHeader_2.54mm:PinHeader_1x01_P2.54mm_Vertical -> TestPoint:TestPoint_Keystone_5015_Micro_Mini
- TP16: value Test Point -> D_OUT2_M; footprint Connector_PinHeader_2.54mm:PinHeader_1x01_P2.54mm_Vertical -> TestPoint:TestPoint_Keystone_5015_Micro_Mini
- TP17: value Test Point -> RTC_CLK; footprint Connector_PinHeader_2.54mm:PinHeader_1x01_P2.54mm_Vertical -> TestPoint:TestPoint_Keystone_5015_Micro_Mini
- TP18: value Test Point -> RTC_EVI; footprint Connector_PinHeader_2.54mm:PinHeader_1x01_P2.54mm_Vertical -> TestPoint:TestPoint_Keystone_5015_Micro_Mini
- TP2: value Test Point -> 3V3; footprint Connector_PinHeader_2.54mm:PinHeader_1x01_P2.54mm_Vertical -> TestPoint:TestPoint_Keystone_5015_Micro_Mini
- TP3: value Test Point -> 5V; footprint Connector_PinHeader_2.54mm:PinHeader_1x01_P2.54mm_Vertical -> TestPoint:TestPoint_Keystone_5015_Micro_Mini
- TP4: value Test Point -> 24V; footprint Connector_PinHeader_2.54mm:PinHeader_1x01_P2.54mm_Vertical -> TestPoint:TestPoint_Keystone_5015_Micro_Mini
- TP5: value Test Point -> VMOD_PG; footprint Connector_PinHeader_2.54mm:PinHeader_1x01_P2.54mm_Vertical -> TestPoint:TestPoint_Keystone_5015_Micro_Mini
- TP6: value Test Point -> VMOD; footprint Connector_PinHeader_2.54mm:PinHeader_1x01_P2.54mm_Vertical -> TestPoint:TestPoint_Keystone_5015_Micro_Mini
- TP7: value Test Point -> VEXT; footprint Connector_PinHeader_2.54mm:PinHeader_1x01_P2.54mm_Vertical -> TestPoint:TestPoint_Keystone_5015_Micro_Mini
- TP8: value Test Point -> VSIM; footprint Connector_PinHeader_2.54mm:PinHeader_1x01_P2.54mm_Vertical -> TestPoint:TestPoint_Keystone_5015_Micro_Mini
- TP9: value Test Point -> VANT; footprint Connector_PinHeader_2.54mm:PinHeader_1x01_P2.54mm_Vertical -> TestPoint:TestPoint_Keystone_5015_Micro_Mini
- moved BT1 110.7 mm to (128.7, 86.2), turned to 0 degrees
- moved TP4 106.9 mm to (121.7, 140.1)
- moved J6 106.0 mm to (138.1, 107.9), turned to 180 degrees
- moved R36 103.3 mm to (142.7, 124.7), turned to 180 degrees
- moved TP11 100.1 mm to (138.7, 132.9), turned to 90 degrees
- moved C23 98.6 mm to (134.8, 121.1), turned to -90 degrees
- moved J4 98.5 mm to (171.4, 100.9), turned to 180 degrees
- moved TP1 98.5 mm to (144.6, 140.1)
- moved SW1 94.5 mm to (142.4, 106.1), turned to 90 degrees
- moved R37 93.7 mm to (153.5, 124.7)
- moved J3 92.1 mm to (146.7, 110.1), turned to 90 degrees
- moved TP12 92.1 mm to (124.7, 112.8), turned to 90 degrees
- moved D7 90.5 mm to (141.7, 118.7)
- moved U3 89.7 mm to (150.9, 97.9), turned to 90 degrees
- moved C24 89.3 mm to (145.6, 121.1), turned to -90 degrees
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Connections:
- J2 pad 4: unconnected-(J2-Pin_4-Pad4) -> GND
Other:
- board size 50 x 80 mm -> 60 x 90 mm
- board text added: "24V"
- board text added: "CodeDog"
- board text added: "POWER"
- board text added: "Powered by"
- board text added: "Remote Sensor Module v1.0"
- board text removed: "3V3"
- board text removed: "VM"

Commit message: FIX: PCB completed.
Parts:
- removed D11, D12: 10V, CodeDog:D_SOD-323
- added Q15: BC817, Package_TO_SOT_SMD:SOT-23, F.Cu at (138.1, 124.1)
- added Q16: BC817, Package_TO_SOT_SMD:SOT-23, F.Cu at (148.9, 124.1)
- added R71: 1k, Resistor_SMD:R_0402_1005Metric_Pad0.72x0.64mm_HandSolder, F.Cu at (136.7, 121.8)
- added R72: 1k, Resistor_SMD:R_0402_1005Metric_Pad0.72x0.64mm_HandSolder, F.Cu at (147.5, 121.8)
- D10, D9: value 1N4148W -> D_Schottky; footprint CodeDog:D_SOD-123 -> Diode_SMD:D_0402_1005Metric
- D4: footprint CodeDog:D_SMA -> CodeDog:D_MiniMELF_Handsoldering
- R36, R37: value 1.8k 0.5W -> 22k; footprint Resistor_SMD:R_0603_1608Metric_Pad0.98x0.95mm_HandSolder -> Resistor_SMD:R_0402_1005Metric_Pad0.72x0.64mm_HandSolder
- R38, R39: value 1k -> 4k7
- R40, R41: value 47k -> 100k
- R50, R51: value 10k -> 100k
- moved J3 28.2 mm to (165.1, 88.8), turned to -90 degrees
- moved R24 17.6 mm to (120.7, 111.6), turned to 0 degrees
- moved Q2 16.0 mm to (122.2, 97.5), turned to -90 degrees
- moved D5 15.7 mm to (124.2, 112.2), turned to 0 degrees
- moved TP12 15.4 mm to (127.9, 97.7), turned to -90 degrees
- moved R31 15.2 mm to (120.0, 109.2), turned to -90 degrees
- moved R32 14.8 mm to (124.4, 97.3)
- moved R30 14.5 mm to (125.4, 97.3), turned to -90 degrees
- moved R28 13.4 mm to (121.1, 100.0), turned to -90 degrees
- moved R25 12.4 mm to (121.9, 109.2), turned to -90 degrees
- moved TP1 12.2 mm to (134.9, 132.7)
- moved C26 11.5 mm to (174.5, 123.5)
- moved R23 11.2 mm to (124.7, 110.0), turned to 0 degrees
- moved C25 11.2 mm to (165.9, 123.5)
- moved R29 10.8 mm to (121.1, 102.3), turned to -90 degrees
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Connections:
- D10 pad 2: GND -> Net-(D10-A)
- D9 pad 2: GND -> Net-(D9-A)
- R36 pad 2: Net-(D9-K) -> Net-(D9-A)
- R37 pad 2: Net-(D10-K) -> Net-(D10-A)
- U6 pad 1: Net-(D9-K) -> Net-(Q15-E)
- U7 pad 1: Net-(D10-K) -> Net-(Q16-E)
Routing:
- net +5V: track 0.00 -> 260.5 mm, vias 0 -> 7
- net +3V3: track 0.00 -> 147.3 mm, vias 0 -> 4
- net +24V: track 0.00 -> 103.3 mm
- net RCS: track 0.00 -> 54.3 mm, vias 0 -> 2
- net D_OUT2_M: track 0.00 -> 49.8 mm, vias 0 -> 2
- net VMOD: track 0.00 -> 47.6 mm, vias 0 -> 5
- net ADC: track 0.00 -> 47.5 mm, vias 0 -> 2
- net A_IN: track 0.00 -> 46.8 mm, vias 0 -> 3
- net D_OUT2: track 0.00 -> 41.8 mm, vias 0 -> 3
- net X_MODEM_WAKE_UP: track 0.00 -> 41.4 mm, vias 0 -> 3
- net D_OUT1_M: track 0.00 -> 39.8 mm, vias 0 -> 2
- net VM: track 0.00 -> 39.6 mm, vias 0 -> 4
- net NRST: track 0.00 -> 37.7 mm, vias 0 -> 2
- net X_MODEM_RX: track 0.00 -> 36.6 mm, vias 0 -> 2
- net D_IN1_M: track 0.00 -> 36.1 mm, vias 0 -> 2
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Other:
- board text added: "Hypersens"
- board text added: "Powered by CodeDog https://www.codedog.pl"
- board text removed: "CodeDog"
- board text removed: "Powered by"

Commit message: FIX: All PCB errors.
Also, LD3905 symbol is changed, to have pin 7 as additional GND required.
Parts:
- D4: footprint CodeDog:D_MiniMELF_Handsoldering -> Diode_SMD:D_MiniMELF_Handsoldering
- D5: footprint CodeDog:D_SOD-123 -> Diode_SMD:D_SOD-123
- moved R28 1.15 mm to (120.0, 100.0)
- moved R29 1.15 mm to (120.0, 102.3)
- moved U1 0.57 mm to (127.0, 117.0)
- moved C15 0.37 mm to (148.4, 107.3)
- moved C16 0.37 mm to (150.2, 107.3)
- moved C13 0.25 mm to (147.7, 104.2)
- moved Q3 0.25 mm to (139.0, 116.2)
- moved Q4 0.25 mm to (149.8, 116.2)
- moved R33 0.25 mm to (121.8, 102.3)
- moved Y1 0.16 mm to (149.4, 104.7)
- moved R16 0.15 mm to (155.6, 104.7)
- moved TP2 0.15 mm to (123.0, 117.5)
- moved C17 0.10 mm to (154.6, 104.7)
- moved C12 0.10 mm to (151.6, 106.5)
- moved J3 0.10 mm to (165.1, 88.7)
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Connections:
- U8 pad 7: (no net) -> GND
Routing:
- net VMOD_VIO: track 6.47 -> 27.3 mm, vias 0 -> 2
- net +3V3: track 147.3 -> 156.6 mm, vias 4 -> 5
- net VSIM: track 19.5 -> 27.8 mm
- net +5V: track 260.5 -> 265.7 mm
- net GND: track 0.00 -> 3.75 mm, vias 0 -> 76
- net Net-(U5-VBACKUP): track 26.4 -> 29.0 mm
- net NRST: track 37.7 -> 40.3 mm
- net Net-(U3B-PB8-BOOT0): track 15.7 -> 17.6 mm
- net DCDC_EN: track 31.6 -> 30.0 mm
- net Net-(Q2-C): track 4.89 -> 6.06 mm
- net VMOD: track 47.6 -> 48.7 mm
- net VMOD_PG: track 8.51 -> 9.58 mm
- net Net-(R42-Pad2): track 2.08 -> 3.08 mm
- net Net-(Q1-G): track 2.67 -> 3.48 mm
