File: KiCad/RS/RS.kicad_pcb (KiCad board)
At the start: 2 copper layers, 60 x 90 mm, 197 parts, among them J1 4.5-28V, J2 Screw_Terminal_01x12, J3 ST-LINK, J4 SPI, J5 MODEM, J6 I2C, J7 GNSS, J8 SIM, J9 ANT., Q1 AO3400A, Q10 BC817, Q11 BC817, Q12 BC817, Q13 BC817, Q14 BC817, Q15 BC817, Q16 BC817, Q2 BC817, Q3 BC817, Q4 BC817, Q5 P60V/2A, Q6 P60V/2A, Q7 BC817, Q8 BC817, Q9 BC817, SW1 SW_Push, U1 MCP1700T-3302E/TT, U10 ST87M01-1301, U11 LDK320M-R, U2 TPS54202, U3 STM32C562KET6, U4 TLP185, U5 RV-3028-C7, U6 TLP185, U7 TLP185, U8 LD39050PUR, U9 EMIF03-SIM02M8, Y1 24MHz CL=8pF ESR=50Ω

Commit message: FIX: New designators synchronized.
Parts:
- renumbered D8 to D10, D13 to D11, D14 to D12, D15 to D13, D16 to D14, D17 to D15, D18 to D16, D19 to D17, D9 to D7, D10 to D8, D7 to D9, Q8 to Q10, Q9 to Q11, Q10 to Q12, Q11 to Q13, Q12 to Q14, Q13 to Q15, Q14 to Q16, Q15 to Q3, Q16 to Q4, Q3 to Q5, Q4 to Q6, Q5 to Q7, Q6 to Q8, Q7 to Q9, R71 to R34, R72 to R35, R34 to R36, R35 to R37, R36 to R38, R37 to R39, R38 to R40, R39 to R41, R40 to R42, R41 to R43, R42 to R44, R43 to R45, R44 to R46, R45 to R47, R46 to R48, R47 to R49, R48 to R50, R49 to R51, R50 to R52, R51 to R53, R52 to R54, R53 to R55, R54 to R56, R55 to R57, R56 to R58, R57 to R59, R58 to R60, R59 to R61, R60 to R62, R61 to R63, R62 to R64, R63 to R65, R64 to R66, R65 to R67, R66 to R68, R67 to R69, R68 to R70, R69 to R71, R70 to R72

Commit message: FIX: Warnings, other.
Routing:
- net SPI_SCK: track 14.8 -> 23.7 mm
- net SPI_MISO: track 21.1 -> 28.9 mm
- net SWDIO: track 13.0 -> 19.3 mm
- net SWO: track 13.8 -> 18.8 mm
- net +3V3: track 156.6 -> 154.2 mm
- net GND: vias 76 -> 101
Other:
- board text added: "DIG. IN1"
- board text added: "DIG. IN2"
- board text added: "DIG. OUT1"
- board text added: "DIG. OUT2"
- board text removed: "DIGITAL IN1"
- board text removed: "DIGITAL IN2"
- board text removed: "DIGITAL OUT1"
- board text removed: "DIGITAL OUT2"
