File: KiCad/RS/nbiot.kicad_sch (KiCad schematic)
At the start: 49 parts, among them J7 GNSS, J8 SIM, J9 ANTENNA, Q10 BC817, Q11 BC817, Q12 BC817, Q9 BC817, U10 ST87M01-1301, U11 LDK320M-R, U8 LD39050PUR, U9 EMIF03-SIM02M8

Commit message: FIX: 0805 to 0402, modem leds+drivers
ADD: Modem part completed!
Parts:
- removed R58, R67, R68, R69: 100k, Resistor_SMD:R_0805_2012Metric_Pad1.20x1.40mm_HandSolder, symbol Device:R
- D17: Mfg Part # B1701USD-20D000114U1930 -> LS R976-NR-1-0-20-R18; URL https://www.digikey.pl/en/products/detail/harvatek-corporat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 -> https://www.digikey.pl/en/products/detail/ams-osram-ag/LS-R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; URL2 CL-270HR-C -> (none)
- D18, D19: Mfg Part # B1701NG--20D000314U1930 -> LG R971-KN-1-0-20-R18; URL https://www.digikey.pl/en/products/detail/harvatek-corporat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 -> https://www.digikey.pl/en/products/detail/ams-osram-ag/LG-R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; URL2 CL-270HR-C -> (none)
- J9: value ANTENNA -> ANT.
- R54: footprint Resistor_SMD:R_0805_2012Metric_Pad1.20x1.40mm_HandSolder -> Resistor_SMD:R_0402_1005Metric_Pad0.72x0.64mm_HandSolder; Mfg Part # ERA-6AEB513V -> RN73R1ETTP5102B25; URL https://www.digikey.pl/en/products/detail/panasonic-industr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 -> https://www.digikey.pl/en/products/detail/koa-speer-electro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
- R55: footprint Resistor_SMD:R_0805_2012Metric_Pad1.20x1.40mm_HandSolder -> Resistor_SMD:R_0402_1005Metric_Pad0.72x0.64mm_HandSolder; Mfg Part # RT0805BRD0724KL -> RT0402BRE0724KL; URL https://www.digikey.pl/en/products/detail/yageo/RT0805BRD07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 -> https://www.digikey.pl/en/products/detail/yageo/RT0402BRE07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
- R56: footprint Resistor_SMD:R_0805_2012Metric_Pad1.20x1.40mm_HandSolder -> Resistor_SMD:R_0402_1005Metric_Pad0.72x0.64mm_HandSolder; Mfg Part # CR0805JB10KS01 -> RMCF0402FT10K0; URL https://www.digikey.pl/en/products/detail/nextgen-component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 -> https://www.digikey.pl/en/products/detail/stackpole-electro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
- R57: footprint Resistor_SMD:R_0805_2012Metric_Pad1.20x1.40mm_HandSolder -> Resistor_SMD:R_0402_1005Metric_Pad0.72x0.64mm_HandSolder; Mfg Part # CR0805JB4K7S01 -> RC0402FR-074K7L; URL https://www.digikey.pl/en/products/detail/nextgen-component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 -> https://www.digikey.pl/en/products/detail/yageo/RC0402FR-07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
- R59, R60, R61: value 470R -> 50Ω; footprint Resistor_SMD:R_0805_2012Metric_Pad1.20x1.40mm_HandSolder -> Resistor_SMD:R_0402_1005Metric_Pad0.72x0.64mm_HandSolder; Mfg Part # CR0805JB470RS1 -> RT0402BRE0750RL; URL https://www.digikey.pl/en/products/detail/nextgen-component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 -> https://www.digikey.pl/en/products/detail/yageo/RT0402BRE07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
- R62: Tolerance (none) -> 0.1%
- R63, R64, R65: value 4k7 -> 2k2; footprint Resistor_SMD:R_0805_2012Metric_Pad1.20x1.40mm_HandSolder -> Resistor_SMD:R_0402_1005Metric_Pad0.72x0.64mm_HandSolder; Mfg Part # CR0805JB4K7S01 -> RMCF0402FT2K20; URL https://www.digikey.pl/en/products/detail/nextgen-component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 -> https://www.digikey.pl/en/products/detail/stackpole-electro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
- R66: value 10k -> 10kΩ; Tolerance (none) -> 0.1%
Other:
- moved on the sheet: Q9, R56, R57, R65

Commit message: FIX: Schematics + BOM.
Parts:
- removed C31: 100n, Capacitor_SMD:C_0805_2012Metric_Pad1.18x1.45mm_HandSolder, symbol Device:C_Small
- removed R56: 10k, Resistor_SMD:R_0402_1005Metric_Pad0.72x0.64mm_HandSolder, symbol Device:R
- added C35: 100n, Capacitor_SMD:C_0402_1005Metric_Pad0.74x0.62mm_HandSolder, symbol Device:C_Small
- added C36: 10μ/10V, Capacitor_SMD:C_0402_1005Metric_Pad0.74x0.62mm_HandSolder, symbol Device:C_Small
- added L6: 120Ω/100MHz/2A, Inductor_SMD:L_0402_1005Metric_Pad0.77x0.64mm_HandSolder, symbol Device:L_Ferrite
- added Q10, Q9: BC817, Package_TO_SOT_SMD:SOT-23, symbol Transistor_BJT:BC817
- added R54: 0R, Resistor_SMD:R_0805_2012Metric_Pad1.20x1.40mm_HandSolder, symbol Device:R
- added R57, R58, R67, R68, R69: 1k, Resistor_SMD:R_0402_1005Metric_Pad0.72x0.64mm_HandSolder, symbol Device:R
- C27: renamed from C23; footprint Capacitor_SMD:C_0805_2012Metric_Pad1.18x1.45mm_HandSolder -> Capacitor_SMD:C_0402_1005Metric_Pad0.74x0.62mm_HandSolder; Mfg Part # CL21B104KBCNNNC -> 0402B104M500CT; URL https://www.digikey.pl/en/products/detail/samsung-electro-m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 -> https://www.digikey.pl/en/products/detail/walsin-technology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
- C28: renamed from C24; footprint Capacitor_SMD:C_0805_2012Metric_Pad1.18x1.45mm_HandSolder -> Capacitor_SMD:C_0402_1005Metric_Pad0.74x0.62mm_HandSolder; Mfg Part # CL21B104KBCNNNC -> 0402B104M500CT; URL https://www.digikey.pl/en/products/detail/samsung-electro-m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 -> https://www.digikey.pl/en/products/detail/walsin-technology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
- C29: renamed from C25; footprint Capacitor_SMD:C_0805_2012Metric_Pad1.18x1.45mm_HandSolder -> Capacitor_SMD:C_0402_1005Metric_Pad0.74x0.62mm_HandSolder; Mfg Part # CL21B104KBCNNNC -> 0402B104M500CT; URL https://www.digikey.pl/en/products/detail/samsung-electro-m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 -> https://www.digikey.pl/en/products/detail/walsin-technology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
- C30: renamed from C26; footprint Capacitor_SMD:C_1206_3216Metric_Pad1.33x1.80mm_HandSolder -> Capacitor_SMD:C_0402_1005Metric_Pad0.74x0.62mm_HandSolder; Mfg Part # GMC31Y5V106Z10NT -> CC0402MRX5R6BB106; URL https://www.digikey.pl/en/products/detail/cal-chip-electron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 -> https://www.digikey.pl/en/products/detail/yageo/CC0402MRX5R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
- C31: renamed from C27; footprint Capacitor_SMD:C_0805_2012Metric_Pad1.18x1.45mm_HandSolder -> Capacitor_SMD:C_0402_1005Metric_Pad0.74x0.62mm_HandSolder; Mfg Part # CL21B104KBCNNNC -> 0402B104M500CT; URL https://www.digikey.pl/en/products/detail/samsung-electro-m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 -> https://www.digikey.pl/en/products/detail/walsin-technology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
- C32: renamed from C28; footprint Capacitor_SMD:C_1206_3216Metric_Pad1.33x1.80mm_HandSolder -> Capacitor_SMD:C_0402_1005Metric_Pad0.74x0.62mm_HandSolder; Mfg Part # GMC31Y5V106Z10NT -> CC0402MRX5R6BB106; URL https://www.digikey.pl/en/products/detail/cal-chip-electron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 -> https://www.digikey.pl/en/products/detail/yageo/CC0402MRX5R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
- C33: renamed from C29; footprint Capacitor_SMD:C_0805_2012Metric_Pad1.18x1.45mm_HandSolder -> Capacitor_SMD:C_0402_1005Metric_Pad0.74x0.62mm_HandSolder; Mfg Part # CL21B104KBCNNNC -> 0402B104M500CT; URL https://www.digikey.pl/en/products/detail/samsung-electro-m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 -> https://www.digikey.pl/en/products/detail/walsin-technology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
- C34: renamed from C30; footprint Capacitor_SMD:C_1206_3216Metric_Pad1.33x1.80mm_HandSolder -> Capacitor_SMD:C_0402_1005Metric_Pad0.74x0.62mm_HandSolder; Mfg Part # GMC31Y5V106Z10NT -> CC0402MRX5R6BB106; URL https://www.digikey.pl/en/products/detail/cal-chip-electron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 -> https://www.digikey.pl/en/products/detail/yageo/CC0402MRX5R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
- C37: renamed from C32; footprint Capacitor_SMD:C_0805_2012Metric_Pad1.18x1.45mm_HandSolder -> Capacitor_SMD:C_0402_1005Metric_Pad0.74x0.62mm_HandSolder; Mfg Part # CL21B104KBCNNNC -> 0402B104M500CT; URL https://www.digikey.pl/en/products/detail/samsung-electro-m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 -> https://www.digikey.pl/en/products/detail/walsin-technology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
- C38: renamed from C33; footprint Capacitor_SMD:C_1206_3216Metric_Pad1.33x1.80mm_HandSolder -> Capacitor_SMD:C_0402_1005Metric_Pad0.74x0.62mm_HandSolder; Mfg Part # GMC31Y5V106Z10NT -> CC0402MRX5R6BB106; URL https://www.digikey.pl/en/products/detail/cal-chip-electron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 -> https://www.digikey.pl/en/products/detail/yageo/CC0402MRX5R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
- C39: renamed from C34; footprint Capacitor_SMD:C_0402_1005Metric -> Inductor_SMD:L_0402_1005Metric_Pad0.77x0.64mm_HandSolder; Mfg Part # C0402C102K1GACAUTO -> C1005C0G1H102J050EA; URL https://www.digikey.pl/en/products/detail/kemet/C0402C102K1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 -> https://www.digikey.pl/en/products/detail/tdk/C1005C0G1H102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
- C40: renamed from C35; footprint Capacitor_SMD:C_0402_1005Metric -> Capacitor_SMD:C_0402_1005Metric_Pad0.74x0.62mm_HandSolder; Mfg Part # CL05C330JB5NNNC -> 0402N330J500CT; URL https://www.digikey.pl/en/products/detail/samsung-electro-m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 -> https://www.digikey.pl/en/products/detail/walsin-technology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
- C41: renamed from C36; value 1μ/50V -> 1μ/10V; footprint Capacitor_SMD:C_0805_2012Metric_Pad1.18x1.45mm_HandSolder -> Capacitor_SMD:C_0402_1005Metric_Pad0.74x0.62mm_HandSolder; Mfg Part # GMC21X7R105K50NT -> NMC0402X5R105K10TRPF; URL https://www.digikey.pl/en/products/detail/cal-chip-electron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 -> https://www.digikey.pl/en/products/detail/nic-components-co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
- J7, J9: MANUFACTURER TE Connectivity -> (none); MAXIMUM_PACKAGE_HEIGHT 1.25 mm -> (none); PARTREV B3 -> (none); STANDARD Manufacturer Recommendations -> (none); URL (none) -> https://www.digikey.pl/en/products/detail/te-connectivity-a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
- L3, L4, L5: footprint Inductor_SMD:L_0805_2012Metric_Pad1.05x1.20mm_HandSolder -> Inductor_SMD:L_0402_1005Metric_Pad0.77x0.64mm_HandSolder; Manufacturer_Part_Number 1-2176744-5 -> (none); Mfg Part # (none) -> WLBD1005HCU121TL; URL (none) -> https://www.digikey.pl/en/products/detail/walsin-technology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
- L7: renamed from L6; footprint Inductor_SMD:L_0805_2012Metric_Pad1.05x1.20mm_HandSolder -> Inductor_SMD:L_0402_1005Metric_Pad0.77x0.64mm_HandSolder; Mfg Part # 1-2176744-5 -> WLBD1005HCU121TL; URL https://www.digikey.pl/en/products/detail/te-connectivity-p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 -> https://www.digikey.pl/en/products/detail/walsin-technology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
- L8: renamed from L7; Mfg Part # LQW15ANR10J0ZD -> WLCM1005Z0JR10TB; URL https://www.digikey.pl/en/products/detail/murata-electronic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 -> https://www.digikey.pl/en/products/detail/walsin-technology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
- R55: renamed from R54; value 51k -> 51k 0.1%; Tolerance (none) -> 0.1%
- R56: renamed from R55; value 24k -> 24k 0.1%; Tolerance (none) -> 0.1%
- R59, R60: value 50Ω -> 4k7; Mfg Part # RT0402BRE0750RL -> RC0402FR-074K7L; URL https://www.digikey.pl/en/products/detail/yageo/RT0402BRE07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 -> https://www.digikey.pl/en/products/detail/yageo/RC0402FR-07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
- R61: value 50Ω -> 1k; Mfg Part # RT0402BRE0750RL -> RNCP0402FTD1K00; URL https://www.digikey.pl/en/products/detail/yageo/RT0402BRE07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 -> https://www.digikey.pl/en/products/detail/stackpole-electro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
- R63, R64, R65: value 2k2 -> 180; Mfg Part # RMCF0402FT2K20 -> CR0402-FX-1800GLF; URL https://www.digikey.pl/en/products/detail/stackpole-electro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 -> https://www.digikey.pl/en/products/detail/bourns-inc/CR0402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
- R66: renamed from R62; value 18k -> 18k 0.1%; footprint Resistor_SMD:R_0805_2012Metric_Pad1.20x1.40mm_HandSolder -> Resistor_SMD:R_0402_1005Metric_Pad0.72x0.64mm_HandSolder; Mfg Part # ERA-6AEB183V -> RN73R1ETTP1802B25; URL https://www.digikey.pl/en/products/detail/panasonic-industr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 -> https://www.digikey.pl/en/products/detail/koa-speer-electro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
- R70: renamed from R66; value 10kΩ -> 10k 0.1%; footprint Resistor_SMD:R_0805_2012Metric_Pad1.20x1.40mm_HandSolder -> Resistor_SMD:R_0402_1005Metric_Pad0.72x0.64mm_HandSolder; Mfg Part # RG2012P-103-B-T5 -> RN04B1002CT10-25; URL https://www.digikey.pl/en/products/detail/susumu/RG2012P-10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 -> https://www.digikey.pl/en/products/detail/cal-chip-electron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
- U10: Mfg Part # (none) -> ST87M01-1301; URL (none) -> https://www.digikey.pl/en/products/detail/stmicroelectronic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
- renumbered Q9 to Q11, Q10 to Q12, Q11 to Q13, Q12 to Q14, R57 to R62
Connections:
- net +5V: now also D17.2 (A), D18.2 (A), D19.2 (A), R54.2; no longer U8.1 (EN), U8.6 (VIN)
- net DCDC_EN: now also R67.1; no longer R63.1
- net GND: now also C35.1, C36.1, Q10.2 (E), Q9.2 (E)
- net MODEM_LED0: now also R68.1; no longer R64.1
- net MODEM_LED1: now also R69.1; no longer R65.1
- net MODEM_WAKE_UP: now also R60.1; no longer U10.39 (WAKE_UP)
- net VMOD: now also L6.1
- net at R61.1: now also Q11.3 (C), U10.38 (RESETn); no longer D19.1 (K)
- net at Q14.3 (C): now also R65.2; no longer R61.2
- net at D17.1 (K): now also R63.1; no longer R59.1
- net at R59.2: now also Q9.1 (B); no longer Q12.3 (C)
- net at Q13.1 (B): now also R68.2; no longer R64.2
- net at R60.2: now also Q10.1 (B); no longer Q13.3 (C)
- net at Q14.1 (B): now also R69.2; no longer R65.2
- net at D18.1 (K): now also R64.1; no longer R60.1
- net at Q12.1 (B): now also R67.2; no longer R63.2
- removed net +3V3: D17.2 (A), D18.2 (A), D19.2 (A), U10.20 (VIO)
- new net: Q9.3 (C), R57.1, U10.39 (WAKE_UP)
- new net: Q12.3 (C), R63.2
- new net: Q13.3 (C), R64.2
- new net: R54.1, U8.1 (EN), U8.6 (VIN)
- new net: D19.1 (K), R65.1
- new net: Q10.3 (C), R58.1, R59.1
- new net VMOD_VIO: C35.2, C36.2, L6.2, R57.2, R58.2, R61.2, U10.20 (VIO)
Other:
- note added: "2.5V 500mA"
- note added: "3V3 200mA"
- moved on the sheet: C29, C30, C31, C32, C33, C34, L3, L4, L5, Q11, R62

Commit message: FIX: Everything. 1.0.
Parts:
- D17: Label (none) -> MP
- D18: Label (none) -> M0
- D19: Label (none) -> M1
Changed lines of the file:
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@@
 	(title_block
 		(title "Remote Sensor Module: NBIOT")
-		(date "2026-07-25")
+		(date "2026-08-15")
 		(rev "0.1")
 		(company "CodeDog")
+		(comment 1 "(c)2026")
+		(comment 2 "All rights reserved")
 	)
 	(text "3V3 200mA"
@@
 			)
 		)
+		(property "Label" "M0"
+			(at 114.3 137.16 0)
+			(hide yes)
+			(show_name no)
+			(do_not_autoplace no)
+			(effects
+				(font
+					(size 1.27 1.27)
+				)
+			)
+		)
 		(pin "1"
 		)
@@
 			)
 		)
+		(property "Label" "MP"
+			(at 63.5 137.16 0)
+			(hide yes)
+			(show_name no)
+			(do_not_autoplace no)
+			(effects
+				(font
+					(size 1.27 1.27)
+				)
+			)
+		)
 		(pin "1"
 		)
@@
 			(at 165.1 137.16 0)
 			(hide yes)
+			(show_name no)
+			(do_not_autoplace no)
+			(effects
+				(font
+					(size 1.27 1.27)
+				)
+			)
+		)
+		(property "Label" "M1"
+			(at 165.1 137.16 0)
+			(hide yes)

Commit message: FIX: All PCB errors.
Also, LD3905 symbol is changed, to have pin 7 as additional GND required.
Connections:
- net GND: now also U8.7 (GND)
Changed lines of the file:
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@@
 	(wire
 		(pts
+			(xy 34.29 46.99) (xy 34.29 50.8)
+		)
+		(stroke
+			(width 0)
+			(type default)
+		)
+	)
+	(wire
+		(pts
 			(xy 19.05 41.91) (xy 21.59 41.91)
 		)
@@
 	)
 	(symbol
+		(lib_id "power:GND")
+		(at 34.29 50.8 0)
+		(unit 1)
+		(body_style 1)
+		(exclude_from_sim no)
+		(in_bom yes)
+		(on_board yes)
+		(in_pos_files yes)
+		(dnp no)
+		(fields_autoplaced yes)
+		(property "Reference" "#PWR0131"
+			(at 34.29 57.15 0)
+			(hide yes)
+			(show_name no)
+			(do_not_autoplace no)
+			(effects
+				(font
+					(size 1.27 1.27)
+				)
+			)
+		)
+		(property "Value" "GND"
+			(at 34.29 55.88 0)
+			(hide yes)
+			(show_name no)
+			(do_not_autoplace no)
+			(effects
+				(font
+					(size 1.27 1.27)
+				)
+			)
+		)
+		(property "Footprint" ""
+			(at 34.29 50.8 0)
+			(hide yes)
+			(show_name no)
+			(do_not_autoplace no)
+			(effects
+				(font
+					(size 1.27 1.27)
+				)
+			)
+		)
+		(property "Datasheet" ""
+			(at 34.29 50.8 0)
+			(hide yes)
+			(show_name no)
+			(do_not_autoplace no)
+			(effects
+				(font
+					(size 1.27 1.27)
+				)
+			)
+		)
+		(property "Description" "Power symbol creates a global label with name \"GND\" , ground"
+			(at 34.29 50.8 0)
+			(hide yes)
+			(show_name no)
+			(do_not_autoplace no)
+			(effects
+				(font
+					(size 1.27 1.27)
+				)
+			)
+		)
+		(pin "1"
+		)
+		(instances
+			(project "RS"
+				(path "/0dbf7561-7a47-4904-aa52-fee53d6c21f5"
+					(reference "#PWR0131")
+					(unit 1)
+				)
+			)
+		)
+	)
+	(symbol
 		(lib_id "Device:R")
 		(at 49.53 46.99 0)
@@
 		(dnp no)
 		(property "Reference" "U8"
-			(at 34.29 45.72 0)
+			(at 20.32 46.99 0)
 			(show_name no)
 			(do_not_autoplace no)
@@
 					(size 1.27 1.27)
 				)
+				(justify left bottom)
 			)
 		)
 		(property "Value" "LD39050PUR"
-			(at 34.29 47.752 0)
+			(at 20.32 47.498 0)
 			(show_name no)
 			(do_not_autoplace no)
@@
 					(size 1.27 1.27)
 				)
+				(justify left top)
 			)
 		)
@@
 		(pin "4"
 		)
+		(pin "7"
+		)
 		(instances
