File: KiCad/RS/nbiot.kicad_sch (KiCad schematic)
At the start: 54 parts, among them J7 GNSS, J8 SIM, J9 ANT., Q10 BC817, Q11 BC817, Q12 BC817, Q13 BC817, Q14 BC817, Q9 BC817, U10 ST87M01-1301, U11 LDK320M-R, U8 LD39050PUR, U9 EMIF03-SIM02M8

Commit message: ADD: UUID fields for all elements.
Parts:
- C27: UUID (none) -> 58ff9971-37b9-4bf4-a752-32300f936261
- C28: UUID (none) -> d853cfa0-55e4-46f1-b19f-3726e9c3f032
- C29: UUID (none) -> a20086d0-6991-439a-8c53-052324fc6bb9
- C30: UUID (none) -> 4db21a40-57ac-45f0-8ac4-f4834601280f
- C31: UUID (none) -> 791b7555-4550-45ca-bb2b-2d52490eaa5e
- C32: UUID (none) -> 1a69015d-f926-4bd6-ab8c-b0d6c0973b26
- C33: UUID (none) -> 4893e8c8-fdc3-4682-ad43-1517cc457e8a
- C34: UUID (none) -> b15ea327-51f7-45ee-94f6-ac8a8fb4e299
- C35: UUID (none) -> 607a9ffb-e46b-45ab-9dd0-7f07bcaf8811
- C36: UUID (none) -> 57c66e25-9836-4ed1-a438-a633bc4f1403
- C37: UUID (none) -> 66dca71c-d826-4f7a-a17f-87d78cdee042
- C38: UUID (none) -> a947a663-9a49-40a6-a712-6018c4aeba14
- C39: UUID (none) -> 6c062791-b6e1-40e9-840d-978410e643c7
- C40: UUID (none) -> ad9df35d-b762-415e-8a05-128784b309bd
- C41: UUID (none) -> 01a79726-82c2-4706-ac42-34c163de7363
- D17: UUID (none) -> e05336d1-d90c-45fe-91c6-e52bec53e546
- D18: UUID (none) -> 0b03ec79-866f-47fa-8adc-239c1220a7de
- D19: UUID (none) -> 93b58d5e-49d1-4a37-8539-f4623fdbbbf1
- J7: UUID (none) -> ad4dc662-e1c3-4920-be49-2924a746ca5b
- J8: UUID (none) -> ae5a1919-a266-4aa3-ac16-a7ff04662812
- J9: UUID (none) -> efee261e-a9e7-411f-b708-6120e68c428d
- L3: UUID (none) -> 45a313c5-fe32-463d-8890-b01fc7bb1a29
- L4: UUID (none) -> bf431453-0691-4632-a333-9ed1b9038fe1
- L5: UUID (none) -> 8ad1336c-65d0-40da-93df-a35e2735025b
- L6: UUID (none) -> 3a653407-f671-40a4-912e-b5601be154a6
- L7: UUID (none) -> af7179fd-cc18-4cd4-91cf-0dfc00c18bc6
- L8: UUID (none) -> 4f102ed5-f379-4199-990f-1e18568660dc
- Q10: UUID (none) -> ac09aeae-88ea-42d3-be61-adb229963053
- Q11: UUID (none) -> d8a3f18b-1aec-4ec3-b223-e1051369cd47
- Q12: UUID (none) -> 09a8b7dc-6b23-4d07-9dc4-e6957dbf6963
- Q13: UUID (none) -> 7b8b2b8c-206b-42e7-b84e-e00ea8747152
- Q14: UUID (none) -> ed929362-ea1c-4245-ad92-b7b095924a51
- Q9: UUID (none) -> 48877e66-56e0-49cf-91ec-d98710e2b09c
- R54: UUID (none) -> 6f9cef16-cff3-4fa8-a07e-2bbd6649dc72
- R55: UUID (none) -> 0307b32f-873d-46cd-b05a-b263aeea5962
- R56: UUID (none) -> bc2eee2c-42c7-4ec9-82ca-277d2c735a59
- R57: UUID (none) -> 5832ba21-97dd-469e-9847-7420135f05fd
- R58: UUID (none) -> 05e3ef6d-1c33-418a-9a21-4be5f8b37a19
- R59: UUID (none) -> 60ce0d49-15a0-4e21-941e-a8e986ad4e85
- R60: UUID (none) -> 782578dc-1404-40c9-b7a7-3a032b280a77
- R61: UUID (none) -> 4fc6c3f1-58fe-4cb3-a6fe-b8ef0db7a856
- R62: UUID (none) -> 6d6a977f-9c2d-4961-93cf-61565d90d217
- R63: UUID (none) -> 4b7ddb8b-35c6-450d-a551-f45877c45eeb
- R64: UUID (none) -> 50c98017-cc06-451f-b67d-0f62c3f5c50d
- R65: UUID (none) -> c7798631-b69e-4afd-b5d6-1e6b6b577827
- R66: UUID (none) -> a85fc91e-39c9-4751-ae3b-5259ba1aad09
- R67: UUID (none) -> 822b76bf-4ced-4d41-945f-00767f745b14
- R68: UUID (none) -> 5a89891f-8a89-4d3f-b8ef-2b04c5e8dae1
- R69: UUID (none) -> a344da58-df28-432d-85cd-2033f0f7db48
- R70: UUID (none) -> 4762b4c7-3bde-4f8b-bf4c-1932f0c1eac1
- U10: UUID (none) -> 510ff453-98c7-4606-b835-1d043bf75a4b
- U10: UUID (none) -> 615bde3b-d4b9-42eb-b4d9-4b56df0dd5b7
- U10: UUID (none) -> 071c1cac-4a69-45d0-a838-cc45e9c41296
- U11: UUID (none) -> 02cd82aa-e46d-49f9-bcbf-cb4a2ba50c54
- U8: UUID (none) -> 7772028d-e8f3-465f-8a96-2a2fec6e010d
- U9: UUID (none) -> 874a0a27-0819-49f7-a4d0-fd8a216e258c

Commit message: FIX: Re-annotate schematics.
Parts:
- renumbered D17 to D15, D18 to D16, D19 to D17, Q9 to Q11, Q10 to Q12, Q11 to Q13, Q12 to Q14, Q13 to Q15, Q14 to Q16, R54 to R56, R55 to R57, R56 to R58, R57 to R59, R58 to R60, R59 to R61, R60 to R62, R61 to R63, R62 to R64, R63 to R65, R64 to R66, R65 to R67, R66 to R68, R67 to R69, R68 to R70, R69 to R71, R70 to R72
