File: KiCad/RS/RS.kicad_sch (KiCad schematic)
At the start: 87 parts, among them J1 XY2500V-B(5.0)-2P, J2 Screw_Terminal_01x12, Q1 AO3400A, Q2 BC817, SW1 SW_Push, U1 MCP1700T-3302E/TT, U2 LM2596S-5, U3 STM32C562KET6, U4 TLP185, U5 RV-3028-C7, Y1 24MHz CL=8pF ESR=50Ω

Commit message: FIX: Schematics + BOM.
Parts:
- removed C2: 470u/50V, Capacitor_THT:CP_Radial_D12.5mm_P5.00mm, symbol Device:C_Polarized_Small
- removed C5, C6: 470u/16V, Capacitor_THT:CP_Radial_D8.0mm_P3.50mm, symbol Device:C_Polarized_Small
- removed D1: LED red, Diode_SMD:D_0805_2012Metric_Pad1.15x1.40mm_HandSolder, symbol Device:LED
- removed D3: SS56, Diode_SMD:D_SMA_Handsoldering, symbol Device:D_Schottky_Filled
- removed R21: 1k, Resistor_SMD:R_0805_2012Metric_Pad1.20x1.40mm_HandSolder, symbol Device:R
- removed R31: 100k, Resistor_SMD:R_0805_2012Metric_Pad1.20x1.40mm_HandSolder, symbol Device:R
- removed U2: LM2596S-5, Package_TO_SOT_SMD:TO-263-5_TabPin3, symbol Regulator_Switching:LM2596S-5
- added C2: 10μ/50V, Capacitor_SMD:C_1210_3225Metric_Pad1.33x2.70mm_HandSolder, symbol Device:C_Small
- added C4, C6: 100n/50V, Capacitor_SMD:C_0402_1005Metric_Pad0.74x0.62mm_HandSolder, symbol Device:C_Small
- added C5: 75pF/50V, Capacitor_SMD:C_0402_1005Metric_Pad0.74x0.62mm_HandSolder, symbol Device:C_Small
- added C7, C8, C9: 10μ/10V, Capacitor_SMD:C_0402_1005Metric_Pad0.74x0.62mm_HandSolder, symbol Device:C_Small
- added D1: SMAJ26A, Diode_SMD:D_SMA, symbol Diode:SMAJ26A
- added D3: LED red, Diode_SMD:D_0805_2012Metric_Pad1.15x1.40mm_HandSolder, symbol Device:LED
- added R24: 120, Resistor_SMD:R_0402_1005Metric_Pad0.72x0.64mm_HandSolder, symbol Device:R
- added R3: 82, Resistor_SMD:R_0402_1005Metric_Pad0.72x0.64mm_HandSolder, symbol Device:R
- added R4: 100k, Resistor_SMD:R_0402_1005Metric_Pad0.72x0.64mm_HandSolder, symbol Device:R
- added R5: 13k3, Resistor_SMD:R_0402_1005Metric_Pad0.72x0.64mm_HandSolder, symbol Device:R
- added U2: TPS54202, Package_TO_SOT_SMD:SOT-23-6, symbol CodeDog:TPS54202DDC
- BT1: MANUFACTURER Keystone -> (none); MAXIMUM_PACKAGE_HEIGHT 3.99mm -> (none); PARTREV D -> (none); SNAPEDA_PN 1056 -> (none); STANDARD Manufacturer Recommendations -> (none)
- C1: value 1μ/50V -> 100n/50V; footprint Capacitor_SMD:C_0805_2012Metric_Pad1.18x1.45mm_HandSolder -> Capacitor_SMD:C_0402_1005Metric_Pad0.74x0.62mm_HandSolder; Mfg Part # GMC21X7R105K50NT -> 0402B104M500CT; URL https://www.digikey.pl/en/products/detail/cal-chip-electron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 -> https://www.digikey.pl/en/products/detail/walsin-technology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
- C11: renamed from C7; footprint Capacitor_SMD:C_0805_2012Metric_Pad1.18x1.45mm_HandSolder -> Capacitor_SMD:C_0402_1005Metric_Pad0.74x0.62mm_HandSolder; Mfg Part # CL21B104KBCNNNC -> 0402B104M500CT; URL https://www.digikey.pl/en/products/detail/samsung-electro-m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 -> https://www.digikey.pl/en/products/detail/walsin-technology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
- C12: renamed from C8; value 1μ/50V -> 1μ/10V; footprint Capacitor_SMD:C_0805_2012Metric_Pad1.18x1.45mm_HandSolder -> Capacitor_SMD:C_0402_1005Metric_Pad0.74x0.62mm_HandSolder; Mfg Part # GMC21X7R105K50NT -> NMC0402X5R105K10TRPF; URL https://www.digikey.pl/en/products/detail/cal-chip-electron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 -> https://www.digikey.pl/en/products/detail/nic-components-co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
- C13: renamed from C9; footprint Capacitor_SMD:C_0805_2012Metric_Pad1.18x1.45mm_HandSolder -> Capacitor_SMD:C_0402_1005Metric_Pad0.74x0.62mm_HandSolder; Mfg Part # CL21B104KBCNNNC -> 0402B104M500CT; URL https://www.digikey.pl/en/products/detail/samsung-electro-m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 -> https://www.digikey.pl/en/products/detail/walsin-technology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
- C14: renamed from C10; footprint Capacitor_SMD:C_0805_2012Metric_Pad1.18x1.45mm_HandSolder -> Capacitor_SMD:C_0402_1005Metric_Pad0.74x0.62mm_HandSolder; Mfg Part # CL21B104KBCNNNC -> 0402B104M500CT; URL https://www.digikey.pl/en/products/detail/samsung-electro-m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 -> https://www.digikey.pl/en/products/detail/walsin-technology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
- C15: renamed from C11; footprint Capacitor_SMD:C_0805_2012Metric_Pad1.18x1.45mm_HandSolder -> Capacitor_SMD:C_0402_1005Metric_Pad0.74x0.62mm_HandSolder; Mfg Part # CML0805C0G120JT50V -> 0402N120J500CT; URL https://www.digikey.pl/en/products/detail/stackpole-electro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 -> https://www.digikey.pl/en/products/detail/walsin-technology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
- C16: renamed from C12; footprint Capacitor_SMD:C_0805_2012Metric_Pad1.18x1.45mm_HandSolder -> Capacitor_SMD:C_0402_1005Metric_Pad0.74x0.62mm_HandSolder; Mfg Part # CML0805C0G120JT50V -> 0402N120J500CT; URL https://www.digikey.pl/en/products/detail/stackpole-electro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 -> https://www.digikey.pl/en/products/detail/walsin-technology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
- C17: renamed from C13; footprint Capacitor_SMD:C_0805_2012Metric_Pad1.18x1.45mm_HandSolder -> Inductor_SMD:L_0402_1005Metric_Pad0.77x0.64mm_HandSolder; Mfg Part # CL21B102KBANNNC -> C1005C0G1H102J050EA; URL https://www.digikey.pl/en/products/detail/samsung-electro-m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 -> https://www.digikey.pl/en/products/detail/tdk/C1005C0G1H102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
- C18: renamed from C14; footprint Capacitor_SMD:C_0805_2012Metric_Pad1.18x1.45mm_HandSolder -> Capacitor_SMD:C_0402_1005Metric_Pad0.74x0.62mm_HandSolder; Mfg Part # CL21B104KBCNNNC -> 0402B104M500CT; URL https://www.digikey.pl/en/products/detail/samsung-electro-m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 -> https://www.digikey.pl/en/products/detail/walsin-technology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
- C19: renamed from C15; value 1μ/50V -> 1μ/10V; footprint Capacitor_SMD:C_0805_2012Metric_Pad1.18x1.45mm_HandSolder -> Capacitor_SMD:C_0402_1005Metric_Pad0.74x0.62mm_HandSolder; Mfg Part # GMC21X7R105K50NT -> NMC0402X5R105K10TRPF; URL https://www.digikey.pl/en/products/detail/cal-chip-electron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 -> https://www.digikey.pl/en/products/detail/nic-components-co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
- C20: renamed from C16; footprint Capacitor_SMD:C_0805_2012Metric_Pad1.18x1.45mm_HandSolder -> Capacitor_SMD:C_0402_1005Metric_Pad0.74x0.62mm_HandSolder; Mfg Part # 0805B225K250CT -> GRM155Z71A225KE44J; URL https://www.digikey.pl/en/products/detail/walsin-technology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 -> https://www.digikey.pl/en/products/detail/murata-electronic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
- C21: renamed from C17; footprint Capacitor_SMD:C_0805_2012Metric_Pad1.18x1.45mm_HandSolder -> Capacitor_SMD:C_0402_1005Metric_Pad0.74x0.62mm_HandSolder; Mfg Part # CL21B104KBCNNNC -> 0402B104M500CT; URL https://www.digikey.pl/en/products/detail/samsung-electro-m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 -> https://www.digikey.pl/en/products/detail/walsin-technology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
- C22: renamed from C18; footprint Capacitor_SMD:C_1206_3216Metric_Pad1.33x1.80mm_HandSolder -> Capacitor_SMD:C_0402_1005Metric_Pad0.74x0.62mm_HandSolder; Mfg Part # GMC31Y5V106Z10NT -> CC0402MRX5R6BB106; URL https://www.digikey.pl/en/products/detail/cal-chip-electron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 -> https://www.digikey.pl/en/products/detail/yageo/CC0402MRX5R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
- C3: value 1μ/50V -> 10μ/50V; footprint Capacitor_SMD:C_0805_2012Metric_Pad1.18x1.45mm_HandSolder -> Capacitor_SMD:C_1210_3225Metric_Pad1.33x2.70mm_HandSolder; Mfg Part # GMC21X7R105K50NT -> 1210B106K500CT; URL https://www.digikey.pl/en/products/detail/cal-chip-electron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 -> https://www.digikey.pl/en/products/detail/walsin-technology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
- D2: Mfg Part # B1701USD-20D000114U1930 -> LS R976-NR-1-0-20-R18; URL https://www.digikey.pl/en/products/detail/harvatek-corporat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 -> https://www.digikey.pl/en/products/detail/ams-osram-ag/LS-R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; URL2 CL-270HR-C -> (none)
- D4: value 3V3 -> 1V; footprint Diode_SMD:D_SOD-523 -> Diode_SMD:D_SMA_Handsoldering; Mfg Part # BZX584B3V3 -> Z1SMA1; URL https://www.digikey.pl/en/products/detail/shenzhen-slkormic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 -> https://www.digikey.pl/en/products/detail/diotec-semiconduc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
- D6: value LED amber -> LED orange; Mfg Part # B1701UY--20D000214U1930 -> LO R976-PS-1-0-20-R18; URL https://www.digikey.pl/en/products/detail/harvatek-corporat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 -> https://www.digikey.pl/en/products/detail/ams-osram-ag/LO-R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; URL2 CL-270HR-C -> (none)
- J1: value XY2500V-B(5.0)-2P -> 4.5-28V; footprint Connector_Phoenix_MSTB:PhoenixContact_MSTBVA_2,5_2-G_1x02_P5.00mm_Vertical -> Connector_Phoenix_MC:PhoenixContact_MCV_1,5_2-G-3.81_1x02_P3.81mm_Vertical
- L1: value 68μH/3.9A -> 15μH/2.05A; footprint Inductor_SMD:L_Coilcraft_MSS1278T-XXX -> Inductor_SMD:L_Cenker_CKCS6045; Mfg Part # SPRH127-680M -> OWINR6045-150; URL (none) -> https://www.digikey.pl/en/products/detail/ole-wolff-electro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
- L2: footprint Inductor_SMD:L_0805_2012Metric_Pad1.05x1.20mm_HandSolder -> Inductor_SMD:L_0402_1005Metric_Pad0.77x0.64mm_HandSolder; Manufacturer_Part_Number HZ0805D102R-10 -> (none); Mfg Part # (none) -> MCB1005B102FBPDG; URL (none) -> https://www.digikey.pl/en/products/detail/inpaq-technology-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
- R1: value 1k -> 49R9; footprint Resistor_SMD:R_0805_2012Metric_Pad1.20x1.40mm_HandSolder -> Resistor_SMD:R_0402_1005Metric_Pad0.72x0.64mm_HandSolder; Mfg Part # CR0805JB1KS001 -> RT0402BRD0749R9L; URL https://www.digikey.pl/en/products/detail/vishay-dale/CRCW0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 -> https://www.digikey.pl/en/products/detail/yageo/RT0402BRD07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
- R11: renamed from R8; now fitted
- R12: renamed from R9; now fitted
- R14: renamed from R11; footprint Resistor_SMD:R_0805_2012Metric_Pad1.20x1.40mm_HandSolder -> Resistor_SMD:R_0402_1005Metric_Pad0.72x0.64mm_HandSolder; Mfg Part # RMC1/10K202FTP -> RT0402FRE072KL; URL https://www.digikey.pl/en/products/detail/kamaya-inc/RMC1-1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 -> https://www.digikey.pl/en/products/detail/yageo/RT0402FRE07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
- R16: renamed from R13; footprint Resistor_SMD:R_0805_2012Metric_Pad1.20x1.40mm_HandSolder -> Resistor_SMD:R_0402_1005Metric_Pad0.72x0.64mm_HandSolder; Mfg Part # RMC1/10K202FTP -> RT0402FRE072KL; URL https://www.digikey.pl/en/products/detail/kamaya-inc/RMC1-1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 -> https://www.digikey.pl/en/products/detail/yageo/RT0402FRE07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
- R2: value 470 -> 180; footprint Resistor_SMD:R_0805_2012Metric_Pad1.20x1.40mm_HandSolder -> Resistor_SMD:R_0402_1005Metric_Pad0.72x0.64mm_HandSolder; Mfg Part # CR0805JB470RS1 -> CR0402-FX-1800GLF; URL https://www.digikey.pl/en/products/detail/nextgen-component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 -> https://www.digikey.pl/en/products/detail/bourns-inc/CR0402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
- R21: renamed from R18; now fitted
- R22: renamed from R19; value 200 -> 120; footprint Resistor_SMD:R_0805_2012Metric_Pad1.20x1.40mm_HandSolder -> Resistor_SMD:R_0402_1005Metric_Pad0.72x0.64mm_HandSolder; Mfg Part # RMCF0805JT200R -> RT0402FRE07120RL; URL https://www.digikey.pl/en/products/detail/stackpole-electro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 -> https://www.digikey.pl/en/products/detail/yageo/RT0402FRE07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
- R23: renamed from R20; Mfg Part # RG2012P-683-B-T5 -> TNPU080568K0BZEA00; TC (none) -> ±5ppm/°C; Tolerance (none) -> 0.1%; URL https://www.digikey.pl/en/products/detail/susumu/RG2012P-68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 -> https://www.digikey.pl/en/products/detail/vishay-dale/TNPU0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
- R25: renamed from R22; value 133R 0.1% -> 133 0.1%; Mfg Part # AR05BTCW1330 -> RQ73C2A133RBTD; TC (none) -> ±10ppm/°C; Tolerance (none) -> 0.1%; URL https://www.digikey.pl/en/products/detail/viking-tech/AR05B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 -> https://www.digikey.pl/en/products/detail/te-connectivity-p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
- R27: renamed from R24; value 100 -> 120; footprint Resistor_SMD:R_0805_2012Metric_Pad1.20x1.40mm_HandSolder -> Resistor_SMD:R_0402_1005Metric_Pad0.72x0.64mm_HandSolder; Mfg Part # CR0805JB100RS1 -> RT0402FRE07120RL; URL https://www.digikey.pl/en/products/detail/nextgen-component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 -> https://www.digikey.pl/en/products/detail/yageo/RT0402FRE07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
- R29: renamed from R26; footprint Resistor_SMD:R_0805_2012Metric_Pad1.20x1.40mm_HandSolder -> Resistor_SMD:R_0402_1005Metric_Pad0.72x0.64mm_HandSolder; Mfg Part # RMCF0805JT200R -> RT0402FRE07200RL; URL https://www.digikey.pl/en/products/detail/stackpole-electro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 -> https://www.digikey.pl/en/products/detail/yageo/RT0402FRE07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
- R30: renamed from R27; value 470 -> 82; footprint Resistor_SMD:R_0805_2012Metric_Pad1.20x1.40mm_HandSolder -> Resistor_SMD:R_0402_1005Metric_Pad0.72x0.64mm_HandSolder; Mfg Part # CR0805JB470RS1 -> RT0402FRE0782RL; URL https://www.digikey.pl/en/products/detail/nextgen-component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 -> https://www.digikey.pl/en/products/detail/yageo/RT0402FRE07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
- R31: renamed from R28; TC (none) -> ±25ppm/°C; Tolerance (none) -> 0.1%
- R33: renamed from R30; footprint Resistor_SMD:R_0805_2012Metric_Pad1.20x1.40mm_HandSolder -> Resistor_SMD:R_0402_1005Metric_Pad0.72x0.64mm_HandSolder; Mfg Part # CR0805JB100KS1 -> RT0402FRE13100KL; URL https://www.digikey.pl/en/products/detail/nextgen-component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 -> https://www.digikey.pl/en/products/detail/yageo/RT0402FRE13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
- R9: renamed from R6; now fitted
- U4: Mfg Part # (none) -> TLP185(GB-TPL,SE; URL (none) -> https://www.digikey.pl/en/products/detail/toshiba-semicondu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
- renumbered C4 to C10, R7 to R10, R10 to R13, R12 to R15, R14 to R17, R15 to R18, R16 to R19, R17 to R20, R23 to R26, R25 to R28, R29 to R32, R3 to R6, R4 to R7, R5 to R8
Connections:
- net +24V: now also C3.1, C2.1, C4.1, D1.1 (A1), U2.3 (VIN); no longer C1.1
- net +3V3: now also R3.2; no longer R2.1
- net +5V: now also R2.1, C6.1, C7.1, C8.1, C9.1; no longer C3.1
- net ADC: now also R24.2
- net GND: now also C2.2, C4.2, C6.2, C7.2, C8.2, C9.2, D1.2 (A2), D3.1 (K), R5.1, U2.1 (GND); no longer C1.2
- net at R23.1, R25.2, R31.2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: now also R24.1
- net at L1.1: now also C1.1, U2.2 (SW)
- net at R1.2: now also C5.1, R4.1
- new net: C1.2, U2.6 (BOOT)
- new net: D3.2 (A), R3.1
- new net: C5.2, R4.2, R5.2, U2.4 (FB)
Other:
- note added: "4.5-28V 0.5A"
- note added: "Max 250mA"
- note added: "Max 2A"
- note removed: "G"
- note removed: "Max 2.5A"
- note removed: "Max 300mA"
- note removed: "POWER"
- moved on the sheet: C10, R30, R32, U1

Commit message: FIX: Everything. 1.0.
Parts:
- D1: footprint Diode_SMD:D_SMA -> CodeDog:D_SMA
- D2: Label (none) -> 5V
- D3: Label (none) -> 3V3
- D4: footprint Diode_SMD:D_SMA_Handsoldering -> CodeDog:D_SMA
- D6: Label (none) -> VM
- TP1: value Test Point -> GND; footprint Connector_PinHeader_2.54mm:PinHeader_1x01_P2.54mm_Vertical -> TestPoint:TestPoint_Keystone_5015_Micro_Mini; now fitted
- TP10: value Test Point -> ADC; footprint Connector_PinHeader_2.54mm:PinHeader_1x01_P2.54mm_Vertical -> TestPoint:TestPoint_Keystone_5015_Micro_Mini; now fitted
- TP11: value Test Point -> RCS; footprint Connector_PinHeader_2.54mm:PinHeader_1x01_P2.54mm_Vertical -> TestPoint:TestPoint_Keystone_5015_Micro_Mini; now fitted
- TP12: value Test Point -> VM; footprint Connector_PinHeader_2.54mm:PinHeader_1x01_P2.54mm_Vertical -> TestPoint:TestPoint_Keystone_5015_Micro_Mini; now fitted
- TP13: value Test Point -> D_IN1_M; footprint Connector_PinHeader_2.54mm:PinHeader_1x01_P2.54mm_Vertical -> TestPoint:TestPoint_Keystone_5015_Micro_Mini; now fitted
- TP14: value Test Point -> D_IN2_M; footprint Connector_PinHeader_2.54mm:PinHeader_1x01_P2.54mm_Vertical -> TestPoint:TestPoint_Keystone_5015_Micro_Mini; now fitted
- TP15: value Test Point -> D_OUT1_M; footprint Connector_PinHeader_2.54mm:PinHeader_1x01_P2.54mm_Vertical -> TestPoint:TestPoint_Keystone_5015_Micro_Mini; now fitted
- TP16: value Test Point -> D_OUT2_M; footprint Connector_PinHeader_2.54mm:PinHeader_1x01_P2.54mm_Vertical -> TestPoint:TestPoint_Keystone_5015_Micro_Mini; now fitted
- TP17: value Test Point -> RTC_CLK; footprint Connector_PinHeader_2.54mm:PinHeader_1x01_P2.54mm_Vertical -> TestPoint:TestPoint_Keystone_5015_Micro_Mini; now fitted
- TP18: value Test Point -> RTC_EVI; footprint Connector_PinHeader_2.54mm:PinHeader_1x01_P2.54mm_Vertical -> TestPoint:TestPoint_Keystone_5015_Micro_Mini; now fitted
- TP2: value Test Point -> 3V3; footprint Connector_PinHeader_2.54mm:PinHeader_1x01_P2.54mm_Vertical -> TestPoint:TestPoint_Keystone_5015_Micro_Mini; now fitted
- TP3: value Test Point -> 5V; footprint Connector_PinHeader_2.54mm:PinHeader_1x01_P2.54mm_Vertical -> TestPoint:TestPoint_Keystone_5015_Micro_Mini; now fitted
- TP4: value Test Point -> 24V; footprint Connector_PinHeader_2.54mm:PinHeader_1x01_P2.54mm_Vertical -> TestPoint:TestPoint_Keystone_5015_Micro_Mini; now fitted
- TP5: value Test Point -> VMOD_PG; footprint Connector_PinHeader_2.54mm:PinHeader_1x01_P2.54mm_Vertical -> TestPoint:TestPoint_Keystone_5015_Micro_Mini; now fitted
- TP6: value Test Point -> VMOD; footprint Connector_PinHeader_2.54mm:PinHeader_1x01_P2.54mm_Vertical -> TestPoint:TestPoint_Keystone_5015_Micro_Mini; now fitted
- TP7: value Test Point -> VEXT; footprint Connector_PinHeader_2.54mm:PinHeader_1x01_P2.54mm_Vertical -> TestPoint:TestPoint_Keystone_5015_Micro_Mini; now fitted
- TP8: value Test Point -> VSIM; footprint Connector_PinHeader_2.54mm:PinHeader_1x01_P2.54mm_Vertical -> TestPoint:TestPoint_Keystone_5015_Micro_Mini; now fitted
- TP9: value Test Point -> VANT; footprint Connector_PinHeader_2.54mm:PinHeader_1x01_P2.54mm_Vertical -> TestPoint:TestPoint_Keystone_5015_Micro_Mini; now fitted
Connections:
- net GND: now also J2.4 (Pin_4)

Commit message: FIX: Schematics and simulation update.
Parts:
- D4: footprint CodeDog:D_SMA -> Diode_SMD:D_MiniMELF_Handsoldering; Mfg Part # Z1SMA1 -> ZMD1; URL https://www.digikey.pl/en/products/detail/diotec-semiconductor/Z1SMA1/22190012 -> https://www.digikey.pl/en/products/detail/diotec-semiconductor/ZMD1/22190996
Changed lines of the file:
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@@
 			)
 		)
-		(property "Footprint" "CodeDog:D_SMA"
+		(property "Footprint" "Diode_SMD:D_MiniMELF_Handsoldering"
 			(at 53.34 161.29 0)
 			(hide yes)
@@
 			)
 		)
-		(property "Mfg Part #" "Z1SMA1"
+		(property "Mfg Part #" "ZMD1"
 			(at 53.34 161.29 0)
 			(hide yes)
@@
 			)
 		)
-		(property "URL" "https://www.digikey.pl/en/products/detail/diotec-semiconductor/Z1SMA1/22190012"
+		(property "URL" "https://www.digikey.pl/en/products/detail/diotec-semiconductor/ZMD1/22190996"
 			(at 53.34 161.29 0)
 			(hide yes)

Commit message: ADD: UUID fields for all elements.
Parts:
- BT1: UUID (none) -> 6c458ca3-8b99-4bff-9a9e-7ed0d44b76fc
- C1: UUID (none) -> c79459f1-3b0c-448c-a7c1-27a51bf198d8
- C10: UUID (none) -> ecd6e28a-82e5-4d6f-9231-ae56ca4fc0cc
- C11: UUID (none) -> 56a2f6d6-0988-4f2e-b7f3-c46e510fd0ee
- C12: UUID (none) -> 039ea6a0-1df1-4546-ae82-063a6626dc7b
- C13: UUID (none) -> 631f3796-2919-42d2-8a97-8c7ed0e5ef7a
- C14: UUID (none) -> 9ea1cd6a-c985-4a87-987f-cd765f7f7647
- C15: UUID (none) -> 2e550da9-66f5-4d78-afa9-d5096db46a83
- C16: UUID (none) -> 298ed757-66c0-4862-ab23-6d6d217285d8
- C17: UUID (none) -> fe037f4b-53e8-4d9e-95a6-486a9cc70590
- C18: UUID (none) -> 485935d7-93ff-4a47-88e6-50e9b157fbf9
- C19: UUID (none) -> ebed36ce-9993-4462-861f-698742554eb4
- C2: UUID (none) -> afbd0ceb-938f-4a9c-8ab6-b7d1c3178570
- C20: UUID (none) -> 829e4cfb-85c2-4176-975a-095c30bd19cb
- C21: UUID (none) -> d63fa10c-6aa2-4532-95bf-e368ab1536ab
- C22: UUID (none) -> 11774a51-ca24-4b90-ae97-3147564de994
- C3: UUID (none) -> 03524bce-0f57-4b02-96f2-ab1692909a27
- C4: UUID (none) -> cd3f3556-f220-4d21-8fbc-7f18b19a09d0
- C5: UUID (none) -> e8463531-59b8-417e-901a-fde19541253d
- C6: UUID (none) -> 586aa043-c939-4181-83f8-b1c2cb390bb6
- C7: UUID (none) -> bafcd414-7a91-4e1a-9684-540ec766bc97
- C8: UUID (none) -> 5277c12a-30da-4702-b90c-2577a3d7ea2b
- C9: UUID (none) -> 968e35f1-1adb-48f6-9508-79262cc4559d
- D1: UUID (none) -> 44ec8d60-77bc-413e-9406-c60d9937a5d0
- D2: UUID (none) -> eeababf0-e948-486b-bc27-1cf8a7f73551
- D3: UUID (none) -> 2b2d2b51-6e0d-4182-8bf9-de66f7cb9d4b
- D4: UUID (none) -> ba3c71b2-825f-42a4-a52b-ae81cf75cc26
- D5: UUID (none) -> dca26f46-ee23-420e-8d27-f117078501bf
- D6: UUID (none) -> cd3bf9bb-faa8-4117-8636-c458e47725fc
- J1: UUID (none) -> 222286fb-d99d-4ebc-b891-9ddc5ac86a80
- J2: UUID (none) -> 4b77fff8-db93-4eee-9147-f2a9246b71e1
- L1: UUID (none) -> 5c454990-2d46-4503-8ce3-957ee93a3b45
- L2: UUID (none) -> 51372508-1d55-458b-a4c9-4a96374f4f8e
- Q1: UUID (none) -> 27b3cfd2-556d-403f-88f7-72eb416db560
- Q2: UUID (none) -> 383435c7-405f-40a2-a682-df3f040c83a8
- R1: UUID (none) -> 0e3ad9e9-0dd5-4c65-9af4-826394ea0e0a
- R10: UUID (none) -> 076ce577-b42c-4ec9-bff3-cde8490f45d6
- R11: UUID (none) -> 36aa9b28-5e36-4901-9efe-5d2b77ffca3c
- R12: UUID (none) -> c0415a31-e9d7-43c5-b3fe-ab847d5de956
- R13: UUID (none) -> 21d4558c-38c9-4190-95e6-b2ab450c4b1d
- R14: UUID (none) -> 23caa2c4-aa20-49d1-90ad-a5ece12399c2
- R15: UUID (none) -> 46be6f16-c53d-4450-ba21-2d6a704dc906
- R16: UUID (none) -> f74285ae-c5f0-472c-8c19-120c2e167b87
- R17: UUID (none) -> 6b1cd494-b6ec-4fbc-b087-c14212c1e359
- R18: UUID (none) -> 8fa54c77-aa16-4e45-afc4-779f07a0babe
- R19: UUID (none) -> 44b24415-2f4f-47fd-8239-d68f2f3c897f
- R2: UUID (none) -> cfac2b4d-f5e9-4bf9-991f-d8a65e8c6d7d
- R20: UUID (none) -> 927c087a-1041-4052-8dea-a184be7aceeb
- R21: UUID (none) -> b356f498-46ba-48a7-b602-6160f43a1da2
- R22: UUID (none) -> 080bfa2c-637b-4a7f-b5dc-dbf5599ea6fd
- R23: UUID (none) -> 133e1206-3406-40ea-bf05-38f4bba0a27e
- R24: UUID (none) -> 46cfcb3a-31b3-4d8a-acff-8bb797226e18
- R25: UUID (none) -> e2034e1b-a26f-42a8-adac-9cd7597339d3
- R26: UUID (none) -> 11b0128e-8fc8-4f30-9733-2c4e3a38e888
- R27: UUID (none) -> e53e5a63-4f19-4d0e-a4ac-0bc155814365
- R28: UUID (none) -> 509a0080-ee54-4906-9552-12a30345083d
- R29: UUID (none) -> d7e69d04-718c-4755-92ef-bc9df42fcd58
- R3: UUID (none) -> 05a46dd6-0990-460b-b880-1ae3cc7645d8
- R30: UUID (none) -> d7983a84-8f95-4eaa-a562-1880c9b7429e
- R31: UUID (none) -> 15c5055f-7443-4b67-9cde-faa6c781b370
- R32: UUID (none) -> 44439e85-5100-405f-acfc-eb4bb76c4400
- R33: UUID (none) -> 88a4cacc-73bb-4dc7-bd20-959e721bcbb9
- R4: UUID (none) -> 476eb679-17cd-45c8-96d7-fda5d5c3746b
- R5: UUID (none) -> 2c7022bf-ea3d-4f99-b631-db1e011395cb
- R6: UUID (none) -> 56f00244-8152-43c6-a124-314333b11a6f
- R7: UUID (none) -> 2878d6d5-1d86-4b3f-8279-6bae178c919d
- R8: UUID (none) -> 1eccdd19-95db-4a74-8d45-8127fb336930
- R9: UUID (none) -> 54748246-8d31-4061-87ac-475755e464e7
- SW1: UUID (none) -> dfe10330-1b8d-4892-8447-62309e139c74
- TP1: UUID (none) -> b0463a9f-7a45-46fa-90a5-6a35394caf0b
- TP10: UUID (none) -> cdee49d1-62d0-458a-8ed6-55a66c46696d
- TP11: UUID (none) -> 943ba74b-df48-4fe7-91e0-4835d3b114f8
- TP12: UUID (none) -> ed04ed14-196f-4d54-99aa-543a896aaa7e
- TP13: UUID (none) -> 91170d39-a7b7-492d-a567-39724bb4e9fe
- TP14: UUID (none) -> 8e2d51b2-f98b-43d8-bffe-931b17d4cc8f
- TP15: UUID (none) -> f50d3988-04bd-4084-a19e-7c6ca4e3b586
- TP16: UUID (none) -> 51e287f7-b78d-4241-85a9-303e5e812aca
- TP17: UUID (none) -> 56495339-108d-47ef-ae10-c12a392b3b97
- TP18: UUID (none) -> f079c7eb-1135-4594-863e-dbc7e0b681d8
- TP2: UUID (none) -> e14df312-870f-4b82-a947-3e7035aa12ec
- TP3: UUID (none) -> e0e772b0-394a-4817-afe2-3d00b689113f
- TP4: UUID (none) -> cf76e336-286d-4f89-817c-657f8af8e1f7
- TP5: UUID (none) -> 9bdfb9aa-35f4-45cf-b3ad-40f5f43f225d
- TP6: UUID (none) -> 8fd7746f-99ad-408b-ada3-cd385643cad6
- TP7: UUID (none) -> 167b6ce3-01a9-4019-942e-4601b3293779
- TP8: UUID (none) -> 8e42096c-9b4e-4f62-8cfc-85abe8803d3b
- TP9: UUID (none) -> 14fd8eaf-b9bd-487b-b7a6-ad196dc02e94
- U1: UUID (none) -> 2758e375-8fcc-4a1c-9c17-5e094a6e4177
- U2: UUID (none) -> c33930ac-2f70-4446-b43c-07d1d78870a2
- U3: UUID (none) -> c89c9e42-33c0-4cab-b295-53b9b6c5ad6f
- U3: UUID (none) -> a7d83ac1-078b-41d6-a1c9-9f5aa3060575
- U4: UUID (none) -> f565444f-c7ba-4b3b-9387-a46861faa8a3
- U5: UUID (none) -> 3a2fae0c-6264-4d04-a2c4-33c75b7549dc
- Y1: UUID (none) -> 7479b9bf-eaea-42f4-b6e4-48112dec9d6c
