File: KiCad/RS/RS.kicad_sch (KiCad schematic)
At the start: 93 parts, among them J1 4.5-28V, J2 Screw_Terminal_01x12, Q1 AO3400A, Q2 BC817, SW1 SW_Push, U1 MCP1700T-3302E/TT, U2 TPS54202, U3 STM32C562KET6, U4 TLP185, U5 RV-3028-C7, Y1 24MHz CL=8pF ESR=50Ω

Commit message: FIX: Warnings, other.
Parts:
- BT1: Mfg Part # (none) -> 1056; now fitted
- TP1, TP10, TP11, TP12, TP13, TP14, TP15, TP16, TP17, TP18, TP2, TP3, TP4, TP5, TP6, TP7, TP8, TP9: Mfg Part # (none) -> 5015; now not fitted

Commit message: FIX: Missing BOM fields.
Parts:
- BT1: URL (none) -> https://www.digikey.pl/en/products/detail/keystone-electron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
Changed lines of the file:
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@@
 			)
 		)
-		(property "Datasheet" ""
+		(property "Datasheet" "https://www.keyelco.com/userAssets/file/K75p2.pdf"
 			(at 217.17 128.27 0)
 			(hide yes)
@@
 			(at 217.17 128.27 0)
 			(hide yes)
+			(show_name no)
+			(do_not_autoplace no)
+			(effects
+				(font
+					(size 1.27 1.27)
+				)
+			)
+		)
+		(property "URL" "https://www.digikey.pl/en/products/detail/keystone-electronics/1056/2020198"
+			(at 217.17 128.27 0)
+			(hide yes)
