File: KiCad/RS/io-connectors.kicad_sch (KiCad schematic)
At the start: 46 parts, among them Q3 FMMT491A, Q4 FMMT491A, Q5 PMV65XP, Q6 PMV65XP, Q7 FMMT491A, Q8 FMMT491A, U6 TLP185, U7 TLP185

Commit message: FIX: BOM, SCH.
Parts:
- removed Q3, Q4, Q7, Q8: FMMT491A, Package_TO_SOT_SMD:SOT-23, symbol CustomSymbols:FMMT491A
- removed Q5, Q6: PMV65XP, PCM_Package_TO_SOT_SMD_AKL:SOT-23, symbol PCM_Transistor_MOSFET_AKL:PMV65XP
- added J3: ST-LINK, Connector_PinHeader_2.54mm:PinHeader_1x06_P2.54mm_Vertical, symbol Connector:Conn_01x06_Pin
- added J4: SPI, Connector_IDC:IDC-Header_2x04_P2.54mm_Vertical_SMD, symbol Connector_Generic:Conn_02x04_Odd_Even
- added J5: MODEM, Connector_PinHeader_2.54mm:PinHeader_1x06_P2.54mm_Vertical, symbol Connector:Conn_01x06_Socket
- added J6: I2C, Connector_PinHeader_2.54mm:PinHeader_1x04_P2.54mm_Vertical, symbol Connector:Conn_01x04_Socket
- added Q3, Q4, Q7, Q8: BC817, Package_TO_SOT_SMD:SOT-23, symbol Transistor_BJT:BC817
- added Q5, Q6: P60V/2A, Package_TO_SOT_SMD:SOT-23W_Handsoldering, symbol Transistor_FET:DMP3099L
- D10, D9: value 1N4148 -> 1N4148W; Mfg Part # (none) -> 1N4148W; URL (none) -> https://www.digikey.pl/en/products/detail/shenzhen-slkormic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
- D11, D12: value BZV55-C10 -> 10V; Mfg Part # BZV55C3V3 -> BZT52B10S; URL (none) -> https://www.digikey.pl/en/products/detail/shenzhen-slkormic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
- D13, D14: value 1N4002 -> 1000V/1A; Mfg Part # (none) -> M7; URL (none) -> https://www.digikey.pl/en/products/detail/diotec-semiconduc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
- D15, D16: value B1701UY--20D000214U1930 -> LED amber; URL (none) -> https://www.digikey.pl/en/products/detail/harvatek-corporat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
- D7, D8: value B1701UY--20D000214U1930 -> LED green; Mfg Part # B1701UY--20D000214U1930 -> B1701NG--20D000314U1930; URL (none) -> https://www.digikey.pl/en/products/detail/harvatek-corporat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
- renumbered R27 to R32, R28 to R33, R29 to R34, R30 to R35, R31 to R36, R32 to R37, R33 to R38, R34 to R39, R35 to R40, R36 to R41, R37 to R42, R38 to R43, R39 to R44, R40 to R45, R41 to R46, R42 to R47, R43 to R48, R44 to R49, R45 to R50, R46 to R51, R47 to R52, R48 to R53
Connections:
- net +3V3: now also J3.1 (Pin_1), J6.2 (Pin_2)
- net +5V: now also J4.8 (Pin_8), J5.2 (Pin_2)
- net D_OUT1: now also Q5.2 (S)
- net D_OUT2: now also Q6.2 (S)
- net GND: now also J3.3 (Pin_3), J4.1 (Pin_1), J4.3 (Pin_3), J5.1 (Pin_1), J6.1 (Pin_1), Q3.2 (E), Q4.2 (E), Q7.2 (E), Q8.2 (E)
- net at R42.2: now also Q5.1 (G)
- net at C21.2, D11.1 (K), D13.1 (K)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: now also Q5.3 (D)
- net at R37.2: now also Q4.1 (B)
- net at C22.2, D12.1 (K), D14.1 (K)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: now also Q6.3 (D)
- net at R46.2, R52.1: now also Q7.1 (B)
- net at R45.2: now also Q8.3 (C)
- net at D8.1 (K): now also Q4.3 (C)
- net at R36.2: now also Q3.1 (B)
- net at D7.1 (K): now also Q3.3 (C)
- net at R43.2: now also Q6.1 (G)
- net at R47.2, R53.1: now also Q8.1 (B)
- net at R44.2: now also Q7.3 (C)
- new net I2C_SCL: J6.4 (Pin_4)
- new net I2C_SDA: J6.3 (Pin_3)
- new net NRST: J3.5 (Pin_5)
- new net SPI_IRQ: J4.7 (Pin_7)
- new net SPI_MISO: J4.5 (Pin_5)
- new net SPI_MOSI: J4.4 (Pin_4)
- new net SPI_NSS: J4.6 (Pin_6)
- new net SPI_SCK: J4.2 (Pin_2)
- new net SWCLK: J3.2 (Pin_2)
- new net SWDIO: J3.4 (Pin_4)
- new net SWO: J3.6 (Pin_6)
- new net X_MODEM_RST: J5.3 (Pin_3)
- new net X_MODEM_RX: J5.5 (Pin_5)
- new net X_MODEM_TX: J5.6 (Pin_6)
- new net X_MODEM_WAKE_UP: J5.4 (Pin_4)
Other:
- note removed: "Y"
- company: (none) -> CodeDog
- title: Remote Sensor Module I/O Sheet -> Remote Sensor Module: Digital I/O Sheet
- moved on the sheet: C19, C20, C21, C22, D10, D11, D12, D13, D14, D9, JP1, JP2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

Commit message: ADD: Connectors placement.
Parts:
- D10, D9: footprint Diode_THT:D_DO-41_SOD81_P10.16mm_Horizontal -> Diode_SMD:D_SOD-123
- D13, D14: footprint Diode_THT:D_DO-41_SOD81_P10.16mm_Horizontal -> Diode_SMD:D_SMA_Handsoldering
Changed lines of the file:
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@@
 			)
 		)
-		(property "Footprint" "Diode_THT:D_DO-41_SOD81_P10.16mm_Horizontal"
+		(property "Footprint" "Diode_SMD:D_SMA_Handsoldering"
 			(at 173.355 106.68 0)
 			(hide yes)
@@
 			)
 		)
-		(property "Footprint" "Diode_THT:D_DO-41_SOD81_P10.16mm_Horizontal"
+		(property "Footprint" "Diode_SMD:D_SOD-123"
 			(at 213.995 60.96 0)
 			(hide yes)
@@
 			)
 		)
-		(property "Footprint" "Diode_THT:D_DO-41_SOD81_P10.16mm_Horizontal"
+		(property "Footprint" "Diode_SMD:D_SMA_Handsoldering"
 			(at 249.555 106.68 0)
 			(hide yes)
@@
 			)
 		)
-		(property "Footprint" "Diode_THT:D_DO-41_SOD81_P10.16mm_Horizontal"
+		(property "Footprint" "Diode_SMD:D_SOD-123"
 			(at 136.525 60.96 0)
 			(hide yes)

Commit message: ADD: RF connections.
Parts:
- JP1, JP2: footprint (none) -> Connector_PinHeader_2.54mm:PinHeader_1x03_P2.54mm_Vertical
Changed lines of the file:
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@@
 			)
 		)
-		(property "Footprint" ""
+		(property "Footprint" "Connector_PinHeader_2.54mm:PinHeader_1x03_P2.54mm_Vertical"
 			(at 185.42 88.9 0)
 			(hide yes)
@@
 			)
 		)
-		(property "Footprint" ""
+		(property "Footprint" "Connector_PinHeader_2.54mm:PinHeader_1x03_P2.54mm_Vertical"
 			(at 261.62 88.9 0)
 			(hide yes)

Commit message: FIX: 0805 to 0402, modem leds+drivers
ADD: Modem part completed!
Parts:
- R32, R33, R50, R51: value 470R -> 470
- R40, R41, R44, R45, R46, R47: footprint Resistor_SMD:R_0805_2012Metric_Pad1.20x1.40mm_HandSolder -> Resistor_SMD:R_0402_1005Metric_Pad0.72x0.64mm_HandSolder; Mfg Part # CR0805JB4K7S01 -> RC0402FR-074K7L; URL https://www.digikey.pl/en/products/detail/nextgen-component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 -> https://www.digikey.pl/en/products/detail/yageo/RC0402FR-07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
- R48, R49, R52, R53: footprint Resistor_SMD:R_0805_2012Metric_Pad1.20x1.40mm_HandSolder -> Resistor_SMD:R_0402_1005Metric_Pad0.72x0.64mm_HandSolder; Mfg Part # CR0805JB10KS01 -> RMCF0402FT10K0; URL https://www.digikey.pl/en/products/detail/nextgen-component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 -> https://www.digikey.pl/en/products/detail/stackpole-electro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
Changed lines of the file:
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@@
 			)
 		)
-		(property "Value" "470R"
+		(property "Value" "470"
 			(at 214.63 125.476 0)
 			(show_name no)
@@
 			)
 		)
-		(property "Footprint" "Resistor_SMD:R_0805_2012Metric_Pad1.20x1.40mm_HandSolder"
+		(property "Footprint" "Resistor_SMD:R_0402_1005Metric_Pad0.72x0.64mm_HandSolder"
 			(at 145.542 128.27 90)
 			(hide yes)
@@
 			)
 		)
-		(property "Datasheet" ""
+		(property "Datasheet" "https://www.seielect.com/catalog/SEI-RMCF_RMCP.pdf"
 			(at 147.32 128.27 0)
 			(hide yes)
@@
 			)
 		)
-		(property "Mfg Part #" "CR0805JB10KS01"
+		(property "Mfg Part #" "RMCF0402FT10K0"
 			(at 147.32 128.27 0)
 			(hide yes)
@@
 			)
 		)
-		(property "URL" "https://www.digikey.pl/en/products/detail/nextgen-components/CR0805JB10KS01/18157959"
+		(property "URL" "https://www.digikey.pl/en/products/detail/stackpole-electronics-inc/RMCF0402FT10K0/1761433"
 			(at 147.32 128.27 0)
 			(hide yes)
@@
 			)
 		)
-		(property "Footprint" "Resistor_SMD:R_0805_2012Metric_Pad1.20x1.40mm_HandSolder"
+		(property "Footprint" "Resistor_SMD:R_0402_1005Metric_Pad0.72x0.64mm_HandSolder"
 			(at 230.632 99.06 90)
 			(hide yes)
@@
 			)
 		)
-		(property "Datasheet" ""
+		(property "Datasheet" "https://yageogroup.com/content/datasheet/asset/file/PYU-RC_GROUP_51_ROHS_L"
 			(at 232.41 99.06 0)
 			(hide yes)
@@
 			)
 		)
-		(property "Mfg Part #" "CR0805JB4K7S01"
+		(property "Mfg Part #" "RC0402FR-074K7L"
 			(at 232.41 99.06 0)
 			(hide yes)
@@
 			)
 		)
-		(property "URL" "https://www.digikey.pl/en/products/detail/nextgen-components/CR0805JB4K7S01/15761328"
+		(property "URL" "https://www.digikey.pl/en/products/detail/yageo/RC0402FR-074K7L/2827563"
 			(at 232.41 99.06 0)
 			(hide yes)
@@
 			)
 		)
-		(property "Footprint" "Resistor_SMD:R_0805_2012Metric_Pad1.20x1.40mm_HandSolder"
+		(property "Footprint" "Resistor_SMD:R_0402_1005Metric_Pad0.72x0.64mm_HandSolder"
 			(at 170.942 123.19 90)
 			(hide yes)
@@
 			)
 		)
-		(property "Datasheet" ""
+		(property "Datasheet" "https://www.seielect.com/catalog/SEI-RMCF_RMCP.pdf"
 			(at 172.72 123.19 0)
 			(hide yes)
@@
 			)
 		)
-		(property "Mfg Part #" "CR0805JB10KS01"
+		(property "Mfg Part #" "RMCF0402FT10K0"
 			(at 172.72 123.19 0)
 			(hide yes)
@@
 			)
 		)
-		(property "URL" "https://www.digikey.pl/en/products/detail/nextgen-components/CR0805JB10KS01/18157959"
+		(property "URL" "https://www.digikey.pl/en/products/detail/stackpole-electronics-inc/RMCF0402FT10K0/1761433"
 			(at 172.72 123.19 0)
 			(hide yes)
@@
 			)
 		)
-		(property "Footprint" "Resistor_SMD:R_0805_2012Metric_Pad1.20x1.40mm_HandSolder"
+		(property "Footprint" "Resistor_SMD:R_0402_1005Metric_Pad0.72x0.64mm_HandSolder"
 			(at 230.632 109.22 90)
 			(hide yes)
@@
 			)
 		)
-		(property "Datasheet" ""
+		(property "Datasheet" "https://yageogroup.com/content/datasheet/asset/file/PYU-RC_GROUP_51_ROHS_L"
 			(at 232.41 109.22 0)
 			(hide yes)
@@
 			)
 		)
-		(property "Mfg Part #" "CR0805JB4K7S01"
+		(property "Mfg Part #" "RC0402FR-074K7L"
 			(at 232.41 109.22 0)
 			(hide yes)
@@
 			)
 		)
-		(property "URL" "https://www.digikey.pl/en/products/detail/nextgen-components/CR0805JB4K7S01/15761328"
+		(property "URL" "https://www.digikey.pl/en/products/detail/yageo/RC0402FR-074K7L/2827563"
 			(at 232.41 109.22 0)
 			(hide yes)
@@
 			)
 		)
-		(property "Value" "470R"
+		(property "Value" "470"
 			(at 138.43 125.476 0)
 			(show_name no)
@@
 			)
 		)
-		(property "Footprint" "Resistor_SMD:R_0805_2012Metric_Pad1.20x1.40mm_HandSolder"
+		(property "Footprint" "Resistor_SMD:R_0402_1005Metric_Pad0.72x0.64mm_HandSolder"
 			(at 218.44 119.888 90)
 			(hide yes)
@@
 			)
 		)
-		(property "Datasheet" ""
+		(property "Datasheet" "https://yageogroup.com/content/datasheet/asset/file/PYU-RC_GROUP_51_ROHS_L"
 			(at 218.44 118.11 0)
 			(hide yes)
@@
 			)
 		)
-		(property "Mfg Part #" "CR0805JB4K7S01"
+		(property "Mfg Part #" "RC0402FR-074K7L"
 			(at 218.44 118.11 0)
 			(hide yes)
@@
 			)
 		)
-		(property "URL" "https://www.digikey.pl/en/products/detail/nextgen-components/CR0805JB4K7S01/15761328"
+		(property "URL" "https://www.digikey.pl/en/products/detail/yageo/RC0402FR-074K7L/2827563"
 			(at 218.44 118.11 90)
 			(hide yes)
@@
 			)
 		)
-		(property "Footprint" "Resistor_SMD:R_0805_2012Metric_Pad1.20x1.40mm_HandSolder"
+		(property "Footprint" "Resistor_SMD:R_0402_1005Metric_Pad0.72x0.64mm_HandSolder"
 			(at 247.142 123.19 90)
 			(hide yes)
@@
 			)
 		)
-		(property "Datasheet" ""
+		(property "Datasheet" "https://www.seielect.com/catalog/SEI-RMCF_RMCP.pdf"
 			(at 248.92 123.19 0)
 			(hide yes)
@@
 			)
 		)
-		(property "Mfg Part #" "CR0805JB10KS01"
+		(property "Mfg Part #" "RMCF0402FT10K0"
 			(at 248.92 123.19 0)
 			(hide yes)
@@
 			)
 		)
-		(property "URL" "https://www.digikey.pl/en/products/detail/nextgen-components/CR0805JB10KS01/18157959"
+		(property "URL" "https://www.digikey.pl/en/products/detail/stackpole-electronics-inc/RMCF0402FT10K0/1761433"
 			(at 248.92 123.19 0)
 			(hide yes)
@@
 			)
 		)
-		(property "Value" "470R"
+		(property "Value" "470"
 			(at 255.27 41.656 90)
 			(show_name no)
@@
 			)
 		)
-		(property "Footprint" "Resistor_SMD:R_0805_2012Metric_Pad1.20x1.40mm_HandSolder"
+		(property "Footprint" "Resistor_SMD:R_0402_1005Metric_Pad0.72x0.64mm_HandSolder"
 			(at 154.432 109.22 90)
 			(hide yes)
@@
 			)
 		)
-		(property "Datasheet" ""
+		(property "Datasheet" "https://yageogroup.com/content/datasheet/asset/file/PYU-RC_GROUP_51_ROHS_L"
 			(at 156.21 109.22 0)
 			(hide yes)
@@
 			)
 		)
-		(property "Mfg Part #" "CR0805JB4K7S01"
+		(property "Mfg Part #" "RC0402FR-074K7L"
 			(at 156.21 109.22 0)
 			(hide yes)
@@
 			)
 		)
-		(property "URL" "https://www.digikey.pl/en/products/detail/nextgen-components/CR0805JB4K7S01/15761328"
+		(property "URL" "https://www.digikey.pl/en/products/detail/yageo/RC0402FR-074K7L/2827563"
 			(at 156.21 109.22 0)
 			(hide yes)
@@
 			)
 		)
-		(property "Footprint" "Resistor_SMD:R_0805_2012Metric_Pad1.20x1.40mm_HandSolder"
+		(property "Footprint" "Resistor_SMD:R_0402_1005Metric_Pad0.72x0.64mm_HandSolder"
 			(at 142.24 119.888 90)
 			(hide yes)
@@
 			)
 		)
-		(property "Datasheet" ""
+		(property "Datasheet" "https://yageogroup.com/content/datasheet/asset/file/PYU-RC_GROUP_51_ROHS_L"
 			(at 142.24 118.11 0)
 			(hide yes)
@@
 			)
 		)
-		(property "Mfg Part #" "CR0805JB4K7S01"
+		(property "Mfg Part #" "RC0402FR-074K7L"
 			(at 142.24 118.11 0)
 			(hide yes)
@@
 			)
 		)
-		(property "URL" "https://www.digikey.pl/en/products/detail/nextgen-components/CR0805JB4K7S01/15761328"
+		(property "URL" "https://www.digikey.pl/en/products/detail/yageo/RC0402FR-074K7L/2827563"
 			(at 142.24 118.11 90)
 			(hide yes)
@@
 			)
 		)
-		(property "Value" "470R"
+		(property "Value" "470"
 			(at 179.07 41.656 90)
 			(show_name no)
@@
 			)
 		)
-		(property "Footprint" "Resistor_SMD:R_0805_2012Metric_Pad1.20x1.40mm_HandSolder"
+		(property "Footprint" "Resistor_SMD:R_0402_1005Metric_Pad0.72x0.64mm_HandSolder"
 			(at 154.432 99.06 90)
 			(hide yes)
@@
 			)
 		)
-		(property "Datasheet" ""
+		(property "Datasheet" "https://yageogroup.com/content/datasheet/asset/file/PYU-RC_GROUP_51_ROHS_L"
 			(at 156.21 99.06 0)
 			(hide yes)
@@
 			)
 		)
-		(property "Mfg Part #" "CR0805JB4K7S01"
+		(property "Mfg Part #" "RC0402FR-074K7L"
 			(at 156.21 99.06 0)
 			(hide yes)
@@
 			)
 		)
-		(property "URL" "https://www.digikey.pl/en/products/detail/nextgen-components/CR0805JB4K7S01/15761328"
+		(property "URL" "https://www.digikey.pl/en/products/detail/yageo/RC0402FR-074K7L/2827563"
 			(at 156.21 99.06 0)
 			(hide yes)
@@
 			)
 		)
-		(property "Footprint" "Resistor_SMD:R_0805_2012Metric_Pad1.20x1.40mm_HandSolder"
+		(property "Footprint" "Resistor_SMD:R_0402_1005Metric_Pad0.72x0.64mm_HandSolder"
 			(at 221.742 128.27 90)
 			(hide yes)
@@
 			)
 		)
-		(property "Datasheet" ""
+		(property "Datasheet" "https://www.seielect.com/catalog/SEI-RMCF_RMCP.pdf"
 			(at 223.52 128.27 0)
 			(hide yes)
@@
 			)
 		)
-		(property "Mfg Part #" "CR0805JB10KS01"
+		(property "Mfg Part #" "RMCF0402FT10K0"
 			(at 223.52 128.27 0)
 			(hide yes)
@@
 			)
 		)
-		(property "URL" "https://www.digikey.pl/en/products/detail/nextgen-components/CR0805JB10KS01/18157959"
+		(property "URL" "https://www.digikey.pl/en/products/detail/stackpole-electronics-inc/RMCF0402FT10K0/1761433"
 			(at 223.52 128.27 0)
 			(hide yes)

Commit message: FIX: Schematics + BOM.
Parts:
- removed C19, C20, C21, C22: 100n, Capacitor_SMD:C_0805_2012Metric_Pad1.18x1.45mm_HandSolder, symbol Device:C_Small
- removed R33, R50, R51: 470, Resistor_SMD:R_0805_2012Metric_Pad1.20x1.40mm_HandSolder, symbol Device:R
- added C23, C24, C25, C26: 100n, Capacitor_SMD:C_0402_1005Metric_Pad0.74x0.62mm_HandSolder, symbol Device:C_Small
- added R41: 47k, Resistor_SMD:R_0402_1005Metric_Pad0.72x0.64mm_HandSolder, symbol Device:R
- D11, D12: footprint Diode_SMD:D_MiniMELF -> Diode_SMD:D_SOD-323
- D15, D16: value LED amber -> LED orange; Mfg Part # B1701UY--20D000214U1930 -> LO R976-PS-1-0-20-R18; URL https://www.digikey.pl/en/products/detail/harvatek-corporat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 -> https://www.digikey.pl/en/products/detail/ams-osram-ag/LO-R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; URL2 CL-270HR-C -> (none)
- D7, D8: Mfg Part # B1701NG--20D000314U1930 -> LG R971-KN-1-0-20-R18; URL https://www.digikey.pl/en/products/detail/harvatek-corporat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 -> https://www.digikey.pl/en/products/detail/ams-osram-ag/LG-R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; URL2 CL-270HR-C -> (none)
- R34: renamed from R32; value 470 -> 180; footprint Resistor_SMD:R_0805_2012Metric_Pad1.20x1.40mm_HandSolder -> Resistor_SMD:R_0402_1005Metric_Pad0.72x0.64mm_HandSolder; Mfg Part # CR0805JB470RS1 -> CR0402-FX-1800GLF; URL https://www.digikey.pl/en/products/detail/nextgen-component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 -> https://www.digikey.pl/en/products/detail/bourns-inc/CR0402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
- R35: value 3k3/0.4W -> 180; footprint Resistor_SMD:R_0805_2012Metric_Pad1.20x1.40mm_HandSolder -> Resistor_SMD:R_0402_1005Metric_Pad0.72x0.64mm_HandSolder; Mfg Part # ESR10EZPJ332 -> CR0402-FX-1800GLF; URL https://www.digikey.pl/en/products/detail/rohm-semiconducto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 -> https://www.digikey.pl/en/products/detail/bourns-inc/CR0402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
- R36: renamed from R34; value 3k3/0.4W -> 1.8k 0.5W; footprint Resistor_SMD:R_0805_2012Metric_Pad1.20x1.40mm_HandSolder -> Resistor_SMD:R_0603_1608Metric_Pad0.98x0.95mm_HandSolder; Mfg Part # ESR10EZPJ332 -> SG73P1JTTD182J; URL https://www.digikey.pl/en/products/detail/rohm-semiconducto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 -> https://www.digikey.pl/en/products/detail/koa-speer-electro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
- R37: value 22k -> 1.8k 0.5W; footprint Resistor_SMD:R_0805_2012Metric_Pad1.20x1.40mm_HandSolder -> Resistor_SMD:R_0603_1608Metric_Pad0.98x0.95mm_HandSolder; Mfg Part # SG73G2ATTD2202D -> SG73P1JTTD182J; URL https://www.digikey.pl/en/products/detail/koa-speer-electronics-inc/SG73G2ATTD2202D/16823265 -> https://www.digikey.pl/en/products/detail/koa-speer-electronics-inc/SG73P1JTTD182J/10189924
- R38: renamed from R36; value 22k -> 1k; footprint Resistor_SMD:R_0805_2012Metric_Pad1.20x1.40mm_HandSolder -> Resistor_SMD:R_0402_1005Metric_Pad0.72x0.64mm_HandSolder; Mfg Part # SG73G2ATTD2202D -> RNCP0402FTD1K00; URL https://www.digikey.pl/en/products/detail/koa-speer-electro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 -> https://www.digikey.pl/en/products/detail/stackpole-electro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
- R39: value 47k -> 1k; footprint Resistor_SMD:R_0805_2012Metric_Pad1.20x1.40mm_HandSolder -> Resistor_SMD:R_0402_1005Metric_Pad0.72x0.64mm_HandSolder; Mfg Part # SFR10EZPJ473 -> RNCP0402FTD1K00; URL https://www.digikey.pl/en/products/detail/rohm-semiconducto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 -> https://www.digikey.pl/en/products/detail/stackpole-electro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
- R40: renamed from R38; footprint Resistor_SMD:R_0805_2012Metric_Pad1.20x1.40mm_HandSolder -> Resistor_SMD:R_0402_1005Metric_Pad0.72x0.64mm_HandSolder; Mfg Part # SFR10EZPJ473 -> RT0402FRE1347KL; URL https://www.digikey.pl/en/products/detail/rohm-semiconducto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 -> https://www.digikey.pl/en/products/detail/yageo/RT0402FRE13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
- R44: renamed from R42; footprint Resistor_SMD:R_0805_2012Metric_Pad1.20x1.40mm_HandSolder -> Resistor_SMD:R_0402_1005Metric_Pad0.72x0.64mm_HandSolder; Mfg Part # CR0805JB1KS001 -> RNCP0402FTD1K00; URL https://www.digikey.pl/en/products/detail/vishay-dale/CRCW0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 -> https://www.digikey.pl/en/products/detail/stackpole-electro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
- R45: renamed from R43; footprint Resistor_SMD:R_0805_2012Metric_Pad1.20x1.40mm_HandSolder -> Resistor_SMD:R_0402_1005Metric_Pad0.72x0.64mm_HandSolder; Mfg Part # CR0805JB1KS001 -> RNCP0402FTD1K00; URL https://www.digikey.pl/en/products/detail/vishay-dale/CRCW0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 -> https://www.digikey.pl/en/products/detail/stackpole-electro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
- R52, R53: value 10k -> 82; Mfg Part # RMCF0402FT10K0 -> RT0402FRE0782RL; URL https://www.digikey.pl/en/products/detail/stackpole-electro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 -> https://www.digikey.pl/en/products/detail/yageo/RT0402FRE07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
- U6, U7: Mfg Part # (none) -> TLP185(GB-TPL,SE; URL (none) -> https://www.digikey.pl/en/products/detail/toshiba-semicondu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
- renumbered R40 to R42, R41 to R43, R44 to R46, R45 to R47, R46 to R48, R47 to R49, R48 to R50, R49 to R51
Connections:
- net +3V3: no longer R34.1
- net +5V: now also R34.1, R35.1
- net D_IN1_M: now also C23.1
- net D_IN2: now also R37.1; no longer R35.1
- net D_IN2_M: now also C24.1, R41.1; no longer R37.1
- net D_OUT1_M: now also R52.2
- net D_OUT2_M: now also R53.2
- net GND: now also C23.2, C24.2, C25.2, C26.2, R41.2; no longer R39.2, R52.2, R53.2
- net at D10.1 (K), U7.1: now also R37.2; no longer R35.2
- net at D16.2 (A): now also R53.1
- net at Q4.1 (B): now also R39.2; no longer R37.2
- net at D12.1 (K), D14.1 (K), JP2.2 (C)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: now also C26.1
- net at D11.1 (K), D13.1 (K), JP1.2 (C)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: now also C25.1
- net at Q7.1 (B), R48.2: no longer R52.1
- net at D15.2 (A): now also R52.1
- net at Q8.1 (B), R49.2: no longer R53.1
- net at D8.2 (A): now also R35.2
Other:
- moved on the sheet: D10, D11, D13, D9, JP1, Q3, Q5, Q7, R34, R36, R38, R40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

Commit message: FIX: Everything. 1.0.
Parts:
- D13, D14: footprint Diode_SMD:D_SMA_Handsoldering -> CodeDog:D_SMA
- D15: Label (none) -> OUT1
- D16: Label (none) -> OUT2
- D7: Label (none) -> IN1
- D8: Label (none) -> IN2
Changed lines of the file:
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@@
 	(title_block
 		(title "Remote Sensor Module: Digital I/O Sheet")
-		(date "2026-07-25")
+		(date "2026-08-15")
 		(rev "0.1")
 		(company "CodeDog")
+		(comment 1 "(c)2026")
+		(comment 2 "All rights reserved")
 	)
 	(junction
@@
 			)
 		)
+		(property "Label" "OUT2"
+			(at 215.9 132.08 0)
+			(hide yes)
+			(show_name no)
+			(do_not_autoplace no)
+			(effects
+				(font
+					(size 1.27 1.27)
+				)
+			)
+		)
 		(pin "1"
 		)
@@
 			)
 		)
+		(property "Label" "IN2"
+			(at 266.7 46.99 0)
+			(hide yes)
+			(show_name no)
+			(do_not_autoplace no)
+			(effects
+				(font
+					(size 1.27 1.27)
+				)
+			)
+		)
 		(pin "1"
 		)
@@
 			)
 		)
+		(property "Label" "OUT1"
+			(at 128.27 132.08 0)
+			(hide yes)
+			(show_name no)
+			(do_not_autoplace no)
+			(effects
+				(font
+					(size 1.27 1.27)
+				)
+			)
+		)
 		(pin "1"
 		)
@@
 			)
 		)
+		(property "Label" "IN1"
+			(at 179.07 46.99 0)
+			(hide yes)
+			(show_name no)
+			(do_not_autoplace no)
+			(effects
+				(font
+					(size 1.27 1.27)
+				)
+			)
+		)
 		(pin "1"
 		)
@@
 			)
 		)
-		(property "Footprint" "Diode_SMD:D_SMA_Handsoldering"
+		(property "Footprint" "CodeDog:D_SMA"
 			(at 161.925 106.68 0)
 			(hide yes)
@@
 			)
 		)
-		(property "Footprint" "Diode_SMD:D_SMA_Handsoldering"
+		(property "Footprint" "CodeDog:D_SMA"
 			(at 249.555 106.68 0)
 			(hide yes)

Commit message: FIX: Schematics and simulation update.
Parts:
- removed D10: 1N4148W, Diode_SMD:D_SOD-123, symbol Diode:1N4002
- removed D11, D12: 10V, Diode_SMD:D_SOD-323, symbol Device:D_Zener
- added D10: D_Schottky, Diode_SMD:D_0402_1005Metric, symbol Device:D_Schottky
- added Q15, Q16: BC817, Package_TO_SOT_SMD:SOT-23, symbol Transistor_BJT:BC817
- added R71, R72: 1k, Resistor_SMD:R_0402_1005Metric_Pad0.72x0.64mm_HandSolder, symbol Device:R
- D9: value 1N4148W -> D_Schottky; footprint Diode_SMD:D_SOD-123 -> Diode_SMD:D_0402_1005Metric; symbol Diode:1N4002 -> Device:D_Schottky; Mfg Part # 1N4148W -> CDBQC0130R-HF; URL https://www.digikey.pl/en/products/detail/shenzhen-slkormic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 -> https://www.digikey.pl/en/products/detail/comchip-technolog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
- R36, R37: value 1.8k 0.5W -> 22k; footprint Resistor_SMD:R_0603_1608Metric_Pad0.98x0.95mm_HandSolder -> Resistor_SMD:R_0402_1005Metric_Pad0.72x0.64mm_HandSolder; Mfg Part # SG73P1JTTD182J -> WR04X2202FTL; URL https://www.digikey.pl/en/products/detail/koa-speer-electro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 -> https://www.digikey.pl/en/products/detail/walsin-technology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
- R38, R39: value 1k -> 4k7; Mfg Part # RNCP0402FTD1K00 -> RC0402FR-074K7L; URL https://www.digikey.pl/en/products/detail/stackpole-electro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 -> https://www.digikey.pl/en/products/detail/yageo/RC0402FR-07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
- R40, R41: value 47k -> 100k; Mfg Part # RT0402FRE1347KL -> (none); URL https://www.digikey.pl/en/products/detail/yageo/RT0402FRE13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 -> (none)
- R50, R51: value 10k -> 100k; Mfg Part # RMCF0402FT10K0 -> RT0402FRE13100KL; URL https://www.digikey.pl/en/products/detail/stackpole-electro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 -> https://www.digikey.pl/en/products/detail/yageo/RT0402FRE13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
Connections:
- net +3V3: now also R71.2, R72.2
- net GND: no longer D9.2 (A)
- net at R37.2: now also D10.2 (A); no longer U7.1
- new net: Q16.3 (C), R72.1
- new net: Q16.2 (E), U7.1
- new net: D10.1 (K), Q16.1 (B)
- new net: Q15.2 (E), U6.1
- new net: D9.1 (K), Q15.1 (B)
- new net: Q15.3 (C), R71.1
- new net: D9.2 (A), R36.2
Other:
- moved on the sheet: D9, R36
