File: KiCad/RS/io-connectors.kicad_sch (KiCad schematic)
At the start: 50 parts, among them J3 ST-LINK, J4 SPI, J5 MODEM, J6 I2C, Q15 BC817, Q16 BC817, Q3 BC817, Q4 BC817, Q5 P60V/2A, Q6 P60V/2A, Q7 BC817, Q8 BC817, U6 TLP185, U7 TLP185

Commit message: ADD: UUID fields for all elements.
Parts:
- C23: UUID (none) -> 2786e63f-0584-4105-9e62-36926e02bd0d
- C24: UUID (none) -> ef01c0f0-6249-45ec-a648-d465adaea5e7
- C25: UUID (none) -> 7a5db7e8-1976-4722-ba81-a6991d2bbdcd
- C26: UUID (none) -> 995e7442-7cd2-4ad2-ba4c-660265688b31
- D10: UUID (none) -> 22a3ec44-3e4b-4cfe-bce1-e3b0c83f1c84
- D13: UUID (none) -> 363c71ff-2c60-4813-9fa3-a55bce40dd2e
- D14: UUID (none) -> 7874ef45-8866-49a5-b780-2dc83989c458
- D15: UUID (none) -> 184ccba5-6855-41f4-8e64-217f763ce0d3
- D16: UUID (none) -> dca864b8-085a-4be7-a52a-e2fe10b56e12
- D7: UUID (none) -> 240572c8-3334-4bf3-83ed-f94d63b9378a
- D8: UUID (none) -> f5712c82-8062-40b6-8005-eb6d9cf9b688
- D9: UUID (none) -> e99d7afb-c0e2-4320-a4db-99471b8d87b0
- J3: UUID (none) -> 7b15bf6e-749d-47f1-b0c7-7cba69b2dcb6
- J4: UUID (none) -> 396247b3-d468-4e95-89f5-7fb1fa3af010
- J5: UUID (none) -> 3b9c8df8-c275-4a98-bee9-936031187a64
- J6: UUID (none) -> 51033af4-040d-4b4c-9bd4-c145d40ac8d1
- JP1: UUID (none) -> 04043d8b-c8c7-4000-8cec-a4e8ed1d01d2
- JP2: UUID (none) -> 5d90d564-8ab7-4c53-869f-a9276faf58fd
- Q15: UUID (none) -> 30df369c-ad82-4e38-9b5e-f1096d1d3f4d
- Q16: UUID (none) -> 3e967478-17ca-4178-a2ab-4e230f303e0c
- Q3: UUID (none) -> 9867d497-2ab6-456f-91b8-7f7029ee8aae
- Q4: UUID (none) -> cbf92398-1f23-49b3-a70f-0b19616667b5
- Q5: UUID (none) -> 71b0764a-4427-479a-9c49-c3e8ff0a222c
- Q6: UUID (none) -> dca3d63c-03a9-4808-a253-187992090688
- Q7: UUID (none) -> d01ec6ae-b263-449b-b34c-142545b5f640
- Q8: UUID (none) -> 0dd18453-0aa6-4e7f-b1bc-55bd4e8e4d9e
- R34: UUID (none) -> 9faf0410-060d-44eb-81e4-e14b5124c438
- R35: UUID (none) -> 0a431c76-b76d-491b-a186-38aa495a6eaa
- R36: UUID (none) -> bf197d5e-1700-4003-9263-338225be7fd3
- R37: UUID (none) -> 9480e89a-290f-4f02-904c-4f402547037a
- R38: UUID (none) -> f505133a-6f41-4dc3-9838-998845bab993
- R39: UUID (none) -> 52f244c2-6172-47de-9ecf-b9659ef74a71
- R40: UUID (none) -> 31365896-20cf-46f8-a53d-125455e6c63f
- R41: UUID (none) -> ddaf66ef-5c55-4c75-8e10-3d4d0fc21a86
- R42: UUID (none) -> 7ee6b8cc-05e4-4507-972e-ff465cb97399
- R43: UUID (none) -> 0fd953de-e4af-4cae-a0bf-42851ea4f981
- R44: UUID (none) -> 41b01bf0-1dcf-4333-bfbd-f9c2a8631f4e
- R45: UUID (none) -> 194c2aa2-8a02-4cb7-87f8-72cbd7ce5ae3
- R46: UUID (none) -> aa565308-9f5c-4bf6-90af-4c98d42f52f6
- R47: UUID (none) -> b012fe7b-179d-4fb9-94dd-a27099674eeb
- R48: UUID (none) -> 33fc4eda-dc6b-4b8d-ac31-ecc6115e88e6
- R49: UUID (none) -> 56b60a1e-3a84-488d-827d-fee4f4118ce7
- R50: UUID (none) -> afc1e850-312d-4cc1-81fd-b4c380eef98d
- R51: UUID (none) -> d86537db-fcaa-42c6-a628-3b711f9a0e1a
- R52: UUID (none) -> 33f1f3c5-b7e3-4d61-9453-97917d6fcfb3
- R53: UUID (none) -> f847ca77-9d51-487d-ba5d-86bba7049910
- R71: UUID (none) -> fd200330-ad85-44c6-b9a1-327ae4e72241
- R72: UUID (none) -> e1e1aa21-61c4-4d80-85b6-781b9811cdca
- U6: UUID (none) -> a749c2c4-d32f-4c12-a5f8-6bc8482217aa
- U7: UUID (none) -> c8eb829e-c090-4c0a-ae8c-47fe46dc549f
