File: KiCad/RS/io-connectors.kicad_sch (KiCad schematic)
At the start: 50 parts, among them J3 ST-LINK, J4 SPI, J5 MODEM, J6 I2C, Q15 BC817, Q16 BC817, Q3 BC817, Q4 BC817, Q5 P60V/2A, Q6 P60V/2A, Q7 BC817, Q8 BC817, U6 TLP185, U7 TLP185

Commit message: FIX: Re-annotate schematics.
Parts:
- renumbered D8 to D10, D13 to D11, D14 to D12, D15 to D13, D16 to D14, D9 to D7, D10 to D8, D7 to D9, Q8 to Q10, Q15 to Q3, Q16 to Q4, Q3 to Q5, Q4 to Q6, Q5 to Q7, Q6 to Q8, Q7 to Q9, R71 to R34, R72 to R35, R34 to R36, R35 to R37, R36 to R38, R37 to R39, R38 to R40, R39 to R41, R40 to R42, R41 to R43, R42 to R44, R43 to R45, R44 to R46, R45 to R47, R46 to R48, R47 to R49, R48 to R50, R49 to R51, R50 to R52, R51 to R53, R52 to R54, R53 to R55

Commit message: FIX: Warnings, other.
Parts:
- J4: now fitted
- R42, R43: Mfg Part # (none) -> RT0402FRE13100KL; URL (none) -> https://www.digikey.pl/en/products/detail/yageo/RT0402FRE13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
Changed lines of the file:
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@@
 			)
 		)
-		(property "Datasheet" ""
+		(property "Datasheet" "https://yageogroup.com/content/datasheet/asset/file/PYU-RT_1-TO-0-01_ROHS_L"
 			(at 153.67 60.96 0)
 			(hide yes)
@@
 			)
 		)
-		(property "Description" "Resistor"
+		(property "Description" "RES 100K OHM 1% 1/16W 0402"
 			(at 153.67 60.96 0)
 			(hide yes)
@@
 			)
 		)
-		(property "Mfg Part #" ""
+		(property "Mfg Part #" "RT0402FRE13100KL"
 			(at 153.67 60.96 0)
 			(hide yes)
@@
 			)
 		)
-		(property "URL" ""
+		(property "URL" "https://www.digikey.pl/en/products/detail/yageo/RT0402FRE13100KL/17018094"
 			(at 153.67 60.96 0)
 			(hide yes)
@@
 			)
 		)
-		(property "Datasheet" ""
+		(property "Datasheet" "https://yageogroup.com/content/datasheet/asset/file/PYU-RT_1-TO-0-01_ROHS_L"
 			(at 241.3 60.96 0)
 			(hide yes)
@@
 			)
 		)
-		(property "Description" "Resistor"
+		(property "Description" "RES 100K OHM 1% 1/16W 0402"
 			(at 241.3 60.96 0)
 			(hide yes)
@@
 			)
 		)
-		(property "Mfg Part #" ""
+		(property "Mfg Part #" "RT0402FRE13100KL"
 			(at 241.3 60.96 0)
 			(hide yes)
@@
 			)
 		)
-		(property "URL" ""
+		(property "URL" "https://www.digikey.pl/en/products/detail/yageo/RT0402FRE13100KL/17018094"
 			(at 241.3 60.96 0)
 			(hide yes)
@@
 		(on_board yes)
 		(in_pos_files yes)
-		(dnp yes)
+		(dnp no)
 		(property "Reference" "J4"
 			(at 74.93 77.978 0)
